File: shematic/bldc_drive/FET_drive.sch (KiCad schematic (older format))
At the start: 40 parts

Commit message: 02.05.2020 01.18 --
Connections:
- net labels added: +12V, +3V3, +V_POW
- net labels removed: VCC, VDD, VSS
Changed lines of the file:
@@
 $Descr A4 11693 8268
 encoding utf-8
-Sheet 3 3
+Sheet 3 4
 Title ""
 Date ""
@@
 $EndComp
 $Comp
-L power:VCC #PWR0103
-U 1 1 5EAD5451
-P 3050 4650
-F 0 "#PWR0103" H 3050 4500 50  0001 C CNN
-F 1 "VCC" H 3067 4823 50  0000 C CNN
-F 2 "" H 3050 4650 50  0001 C CNN
-F 3 "" H 3050 4650 50  0001 C CNN
-	1    3050 4650
-	1    0    0    -1
-$EndComp
-$Comp
-L power:VCC #PWR0104
-U 1 1 5EAD5A9B
-P 3050 3100
-F 0 "#PWR0104" H 3050 2950 50  0001 C CNN
-F 1 "VCC" H 3067 3273 50  0000 C CNN
-F 2 "" H 3050 3100 50  0001 C CNN
-F 3 "" H 3050 3100 50  0001 C CNN
-	1    3050 3100
-	1    0    0    -1
-$EndComp
-$Comp
 L power:GND #PWR0105
 U 1 1 5EAD60E9
@@
 Wire Wire Line
 	3050 3150 3050 3100
-$Comp
-L power:VCC #PWR0108
-U 1 1 5EAD9DE2
-P 3050 1400
-F 0 "#PWR0108" H 3050 1250 50  0001 C CNN
-F 1 "VCC" H 3067 1573 50  0000 C CNN
-F 2 "" H 3050 1400 50  0001 C CNN
-F 3 "" H 3050 1400 50  0001 C CNN
-	1    3050 1400
-	1    0    0    -1
-$EndComp
 Wire Wire Line
 	3050 1450 3050 1400
@@
 Wire Wire Line
 	3400 4650 3050 4650
-Connection ~ 3050 4650
 Wire Wire Line
 	3400 3100 3050 3100
-Connection ~ 3050 3100
 Wire Wire Line
 	3400 1400 3050 1400
-Connection ~ 3050 1400
 $Comp
 L Device:CP C?
@@
 	1    0    0    -1
 $EndComp
-$Comp
-L power:VCC #PWR?
-U 1 1 5EB37945
-P 4750 6300
-F 0 "#PWR?" H 4750 6150 50  0001 C CNN
-F 1 "VCC" H 4767 6473 50  0000 C CNN
-F 2 "" H 4750 6300 50  0001 C CNN
-F 3 "" H 4750 6300 50  0001 C CNN
-	1    4750 6300
-	1    0    0    -1
-$EndComp
-Wire Wire Line
-	4750 6300 4750 6450
 Wire Wire Line
 	4750 6750 4750 6950
@@
 Wire Wire Line
 	8050 1650 8050 2550
-Connection ~ 8050 1650
-$Comp
-L power:VSS #PWR?
-U 1 1 5EBCA6DE
-P 8050 1050
-F 0 "#PWR?" H 8050 900 50  0001 C CNN
-F 1 "VSS" H 8067 1223 50  0000 C CNN
-F 2 "" H 8050 1050 50  0001 C CNN
-F 3 "" H 8050 1050 50  0001 C CNN
-	1    8050 1050
-	1    0    0    -1
-$EndComp
-Wire Wire Line
-	8050 1050 8050 1650
-$Comp
-L power:VDD #PWR?
-U 1 1 5EBCE6E6
-P 7000 1200
-F 0 "#PWR?" H 7000 1050 50  0001 C CNN
-F 1 "VDD" H 7017 1373 50  0000 C CNN
-F 2 "" H 7000 1200 50  0001 C CNN
-F 3 "" H 7000 1200 50  0001 C CNN
-	1    7000 1200
-	1    0    0    -1
-$EndComp
-Wire Wire Line
-	7000 1200 7000 1450
 $Comp
 L power:GND #PWR?
@@
 Text GLabel 5850 1750 0    50   Input ~ 0
 CURRENT_SENSE
+Text GLabel 8050 1100 1    50   Input ~ 0
++V_POW
+Wire Wire Line
+	8050 1100 8050 1650
+Connection ~ 8050 1650
+$Comp
+L power:+3V3 #PWR?
+U 1 1 5EAEC5E3
+P 7000 1050
+F 0 "#PWR?" H 7000 900 50  0001 C CNN
+F 1 "+3V3" H 7015 1223 50  0000 C CNN
+F 2 "" H 7000 1050 50  0001 C CNN
+F 3 "" H 7000 1050 50  0001 C CNN
+	1    7000 1050
+	1    0    0    -1
+$EndComp
+Wire Wire Line
+	7000 1050 7000 1450
+$Comp
+L power:+12V #PWR?
+U 1 1 5EAF355D
+P 4750 6200
+F 0 "#PWR?" H 4750 6050 50  0001 C CNN
+F 1 "+12V" H 4765 6373 50  0000 C CNN
+F 2 "" H 4750 6200 50  0001 C CNN
+F 3 "" H 4750 6200 50  0001 C CNN
+	1    4750 6200
+	1    0    0    -1
+$EndComp
+$Comp
+L power:+12V #PWR?
+U 1 1 5EAF4118
+P 3050 4650
+F 0 "#PWR?" H 3050 4500 50  0001 C CNN
+F 1 "+12V" H 3065 4823 50  0000 C CNN
+F 2 "" H 3050 4650 50  0001 C CNN
+F 3 "" H 3050 4650 50  0001 C CNN
+	1    3050 4650
+	1    0    0    -1
+$EndComp
+Connection ~ 3050 4650
+$Comp
+L power:+12V #PWR?
+U 1 1 5EAF4973
+P 3050 3100
+F 0 "#PWR?" H 3050 2950 50  0001 C CNN
+F 1 "+12V" H 3065 3273 50  0000 C CNN
+F 2 "" H 3050 3100 50  0001 C CNN
+F 3 "" H 3050 3100 50  0001 C CNN
+	1    3050 3100
+	1    0    0    -1
+$EndComp
+Connection ~ 3050 3100
+$Comp
+L power:+12V #PWR?
+U 1 1 5EAF4C3A
+P 3050 1400
+F 0 "#PWR?" H 3050 1250 50  0001 C CNN
+F 1 "+12V" H 3065 1573 50  0000 C CNN
+F 2 "" H 3050 1400 50  0001 C CNN
+F 3 "" H 3050 1400 50  0001 C CNN
+	1    3050 1400
+	1    0    0    -1
+$EndComp
+Connection ~ 3050 1400
+Wire Wire Line
+	4750 6200 4750 6450
 $EndSCHEMATC

Commit message: 10.05.2020 21.40 --
Parts:
- added C?: 1u, symbol Device:C
- added D?: DZ2S033X0L, Diode_SMD:D_SOD-523, symbol Diode:DZ2S033X0L
- added R?: 10k, symbol Device:R
- added R?: 1k, symbol Device:R
Connections:
- net +V_POW: now also R?.2
- net GND: now also C?.2, D?.2 (A), R?.1
- new net V_POW_MEAS: C?.1, D?.1 (K), R?.1, R?.2
Other:
- moved on the sheet: C?
Changed lines of the file:
@@
 L power:GND #PWR0101
 U 1 1 5EAD00DD
-P 4750 6950
-F 0 "#PWR0101" H 4750 6700 50  0001 C CNN
-F 1 "GND" H 4755 6777 50  0000 C CNN
-F 2 "" H 4750 6950 50  0001 C CNN
-F 3 "" H 4750 6950 50  0001 C CNN
-	1    4750 6950
+P 3800 6950
+F 0 "#PWR0101" H 3800 6700 50  0001 C CNN
+F 1 "GND" H 3805 6777 50  0000 C CNN
+F 2 "" H 3800 6950 50  0001 C CNN
+F 3 "" H 3800 6950 50  0001 C CNN
+	1    3800 6950
 	1    0    0    -1
 $EndComp
@@
 L Device:CP C?
 U 1 1 5EB36141
-P 4750 6600
-F 0 "C?" H 4868 6646 50  0000 L CNN
-F 1 "47 uF 35V" H 4868 6555 50  0000 L CNN
-F 2 "" H 4788 6450 50  0001 C CNN
-F 3 "~" H 4750 6600 50  0001 C CNN
-	1    4750 6600
-	1    0    0    -1
-$EndComp
-Wire Wire Line
-	4750 6750 4750 6950
+P 3800 6600
+F 0 "C?" H 3918 6646 50  0000 L CNN
+F 1 "47 uF 35V" H 3918 6555 50  0000 L CNN
+F 2 "" H 3838 6450 50  0001 C CNN
+F 3 "~" H 3800 6600 50  0001 C CNN
+	1    3800 6600
+	1    0    0    -1
+$EndComp
+Wire Wire Line
+	3800 6750 3800 6950
 $Comp
 L Device:R R?
@@
 L power:+12V #PWR?
 U 1 1 5EAF355D
-P 4750 6200
-F 0 "#PWR?" H 4750 6050 50  0001 C CNN
-F 1 "+12V" H 4765 6373 50  0000 C CNN
-F 2 "" H 4750 6200 50  0001 C CNN
-F 3 "" H 4750 6200 50  0001 C CNN
-	1    4750 6200
+P 3800 6200
+F 0 "#PWR?" H 3800 6050 50  0001 C CNN
+F 1 "+12V" H 3815 6373 50  0000 C CNN
+F 2 "" H 3800 6200 50  0001 C CNN
+F 3 "" H 3800 6200 50  0001 C CNN
+	1    3800 6200
 	1    0    0    -1
 $EndComp
@@
 Connection ~ 3050 1400
 Wire Wire Line
-	4750 6200 4750 6450
+	3800 6200 3800 6450
+$Comp
+L Device:R R?
+U 1 1 5EBDD289
+P 5000 6200
+AR Path="/5EB1ABF5/5EBDD289" Ref="R?"  Part="1"
+AR Path="/5EACE430/5EBDD289" Ref="R?"  Part="1"
+F 0 "R?" H 4930 6154 50  0000 R CNN
+F 1 "10k" H 4930 6245 50  0000 R CNN
+F 2 "" V 4930 6200 50  0001 C CNN
+F 3 "~" H 5000 6200 50  0001 C CNN
+	1    5000 6200
+	-1   0    0    1
+$EndComp
+$Comp
+L Device:R R?
+U 1 1 5EBDD28F
+P 5000 6600
+AR Path="/5EB1ABF5/5EBDD28F" Ref="R?"  Part="1"
+AR Path="/5EACE430/5EBDD28F" Ref="R?"  Part="1"
+F 0 "R?" H 4930 6554 50  0000 R CNN
+F 1 "1k" H 4930 6645 50  0000 R CNN
+F 2 "" V 4930 6600 50  0001 C CNN
+F 3 "~" H 5000 6600 50  0001 C CNN
+	1    5000 6600
+	-1   0    0    1
+$EndComp
+$Comp
+L Diode:DZ2S033X0L D?
+U 1 1 5EBDD295
+P 4750 6600
+AR Path="/5EB1ABF5/5EBDD295" Ref="D?"  Part="1"
+AR Path="/5EACE430/5EBDD295" Ref="D?"  Part="1"
+F 0 "D?" V 4650 6450 50  0000 L CNN
+F 1 "DZ2S033X0L" V 5250 6450 50  0001 L CNN
+F 2 "Diode_SMD:D_SOD-523" H 4750 6425 50  0001 C CNN
+F 3 "https://industrial.panasonic.com/content/data/SC/ds/ds4/DZ2S03300L_E.pdf" H 4750 6600 50  0001 C CNN
+	1    4750 6600
+	0    1    1    0
+$EndComp
+$Comp
+L Device:C C?
+U 1 1 5EBDD29B
+P 5250 6600
+AR Path="/5EB1ABF5/5EBDD29B" Ref="C?"  Part="1"
+AR Path="/5EACE430/5EBDD29B" Ref="C?"  Part="1"
+F 0 "C?" H 5365 6646 50  0000 L CNN
+F 1 "1u" H 5365 6555 50  0000 L CNN
+F 2 "" H 5288 6450 50  0001 C CNN
+F 3 "~" H 5250 6600 50  0001 C CNN
+	1    5250 6600
+	1    0    0    -1
+$EndComp
+$Comp
+L power:GND #PWR?
+U 1 1 5EBDD2A1
+P 5000 6950
+AR Path="/5EB1ABF5/5EBDD2A1" Ref="#PWR?"  Part="1"
+AR Path="/5EACE430/5EBDD2A1" Ref="#PWR?"  Part="1"
+F 0 "#PWR?" H 5000 6700 50  0001 C CNN
+F 1 "GND" H 5005 6777 50  0000 C CNN
+F 2 "" H 5000 6950 50  0001 C CNN
+F 3 "" H 5000 6950 50  0001 C CNN
+	1    5000 6950
+	1    0    0    -1
+$EndComp
+Wire Wire Line
+	4750 6750 4750 6850
+Wire Wire Line
+	4750 6850 5000 6850
+Wire Wire Line
+	5250 6850 5250 6750
+Wire Wire Line
+	5000 6950 5000 6850
+Connection ~ 5000 6850
+Wire Wire Line
+	5000 6850 5250 6850
+Wire Wire Line
+	5000 6750 5000 6850
+Wire Wire Line
+	5000 6450 5000 6400
+Wire Wire Line
+	4750 6450 4750 6400
+Wire Wire Line
+	4750 6400 5000 6400
+Connection ~ 5000 6400
+Wire Wire Line
+	5000 6400 5000 6350
+Wire Wire Line
+	5250 6450 5250 6400
+Wire Wire Line
+	5250 6400 5000 6400
+Text GLabel 5000 5850 1    50   Input ~ 0
++V_POW
+Wire Wire Line
+	5000 6050 5000 5850
+Text GLabel 5500 6400 2    50   Input ~ 0
+V_POW_MEAS
+Wire Wire Line
+	5500 6400 5250 6400
+Connection ~ 5250 6400
+$Comp
+L power:+12V #PWR?
+U 1 1 5EC00656
+P 5100 4300
+F 0 "#PWR?" H 5100 4150 50  0001 C CNN
+F 1 "+12V" H 5115 4473 50  0000 C CNN
+F 2 "" H 5100 4300 50  0001 C CNN
+F 3 "" H 5100 4300 50  0001 C CNN
+	1    5100 4300
+	1    0    0    -1
+$EndComp
 $EndSCHEMATC
