File: shematic/bldc_drive/FET_drive.sch (KiCad schematic (older format))
At the start: 44 parts

Commit message: 22.05.2020 21.40 --
Parts:
- gave numbers to parts that had none: 44

Commit message: 03.06.2020 21.40 --
Parts:
- Q1, Q2, Q3, Q4, Q5, Q6, Q7: value IRF540N -> IRF1407
Changed lines of the file:
@@
 $Descr A4 11693 8268
 encoding utf-8
-Sheet 3 5
+Sheet 3 6
 Title ""
 Date ""
@@
 P 7950 5450
 F 0 "Q5" H 8154 5496 50  0000 L CNN
-F 1 "IRF540N" H 8154 5405 50  0000 L CNN
+F 1 "IRF1407" H 8154 5405 50  0000 L CNN
 F 2 "Package_TO_SOT_THT:TO-220-3_Vertical" H 8200 5375 50  0001 L CIN
 F 3 "http://www.irf.com/product-info/datasheets/data/irf540n.pdf" H 7950 5450 50  0001 L CNN
@@
 P 9350 4450
 F 0 "Q7" H 9554 4496 50  0000 L CNN
-F 1 "IRF540N" H 9554 4405 50  0000 L CNN
+F 1 "IRF1407" H 9554 4405 50  0000 L CNN
 F 2 "Package_TO_SOT_THT:TO-220-3_Vertical" H 9600 4375 50  0001 L CIN
 F 3 "http://www.irf.com/product-info/datasheets/data/irf540n.pdf" H 9350 4450 50  0001 L CNN
@@
 P 9350 3450
 F 0 "Q6" H 9554 3496 50  0000 L CNN
-F 1 "IRF540N" H 9554 3405 50  0000 L CNN
+F 1 "IRF1407" H 9554 3405 50  0000 L CNN
 F 2 "Package_TO_SOT_THT:TO-220-3_Vertical" H 9600 3375 50  0001 L CIN
 F 3 "http://www.irf.com/product-info/datasheets/data/irf540n.pdf" H 9350 3450 50  0001 L CNN
@@
 P 7950 4500
 F 0 "Q4" H 8100 4400 50  0000 L CNN
-F 1 "IRF540N" H 8100 4300 50  0000 L CNN
+F 1 "IRF1407" H 8100 4300 50  0000 L CNN
 F 2 "Package_TO_SOT_THT:TO-220-3_Vertical" H 8200 4425 50  0001 L CIN
 F 3 "http://www.irf.com/product-info/datasheets/data/irf540n.pdf" H 7950 4500 50  0001 L CNN
@@
 P 7950 3450
 F 0 "Q3" H 8100 3350 50  0000 L CNN
-F 1 "IRF540N" H 8100 3250 50  0000 L CNN
+F 1 "IRF1407" H 8100 3250 50  0000 L CNN
 F 2 "Package_TO_SOT_THT:TO-220-3_Vertical" H 8200 3375 50  0001 L CIN
 F 3 "http://www.irf.com/product-info/datasheets/data/irf540n.pdf" H 7950 3450 50  0001 L CNN
@@
 P 6400 4550
 F 0 "Q2" H 6604 4596 50  0000 L CNN
-F 1 "IRF540N" H 6604 4505 50  0000 L CNN
+F 1 "IRF1407" H 6604 4505 50  0000 L CNN
 F 2 "Package_TO_SOT_THT:TO-220-3_Vertical" H 6650 4475 50  0001 L CIN
 F 3 "http://www.irf.com/product-info/datasheets/data/irf540n.pdf" H 6400 4550 50  0001 L CNN
@@
 P 6400 3450
 F 0 "Q1" H 6604 3496 50  0000 L CNN
-F 1 "IRF540N" H 6604 3405 50  0000 L CNN
+F 1 "IRF1407" H 6604 3405 50  0000 L CNN
 F 2 "Package_TO_SOT_THT:TO-220-3_Vertical" H 6650 3375 50  0001 L CIN
 F 3 "http://www.irf.com/product-info/datasheets/data/irf540n.pdf" H 6400 3450 50  0001 L CNN

Commit message: 11.06.2020 21.40 --
Parts:
- added D7: 1N4148WS, Diode_SMD:D_SOD-123, symbol Diode:1N4148WS
- added Q10: BC807, Package_TO_SOT_SMD:SOT-23, symbol Transistor_BJT:BC807
- added Q9: BC817, Package_TO_SOT_SMD:SOT-23, symbol Transistor_BJT:BC817
- added R35: 1k, Resistor_SMD:R_0603_1608Metric, symbol Device:R
- C10, C11, C9: footprint (none) -> Capacitor_Tantalum_SMD:CP_EIA-6032-28_Kemet-C
- C12: footprint (none) -> Capacitor_SMD:C_Elec_8x6.2
- C13: footprint (none) -> Capacitor_SMD:C_0805_2012Metric
- D2, D3, D4: footprint Diode_SMD:D_SOD-323 -> Diode_SMD:D_SOD-123
- R10, R11, R12, R13, R14, R15, R8, R9: footprint (none) -> Resistor_SMD:R_0603_1608Metric
- R16, R17, R18, R19, R20, R21, R22, R24, R25, R26, R28, R29, R30, R31: footprint (none) -> Resistor_SMD:R_0805_2012Metric
- R23: value 1k -> 560R; footprint (none) -> Resistor_SMD:R_0805_2012Metric
- R27: footprint (none) -> Resistor_SMD:R_2512_6332Metric
- U6, U7, U8: footprint (none) -> Package_SO:SOIC-8-1EP_3.9x4.9mm_P1.27mm_EP2.29x3mm
Connections:
- net +12V: now also Q10.2 (E)
- net GND: now also Q9.2 (E)
- net LOCK_H: now also D7.2 (A); no longer R23.2
- new net: Q10.1 (B), Q9.3 (C)
- new net: Q9.1 (B), R35.1
- new net: D7.1 (K), R35.2
- new net Lock_S: Q10.3 (C), R23.2
Other:
- moved on the sheet: C12, C13, D5, R14, R15

Commit message: --
Parts:
- R27: footprint Resistor_SMD:R_2512_6332Metric -> Resistor_SMD:R_4020_10251Metric_Pad1.65x5.30mm_HandSolder
- U6, U7, U8: footprint Package_SO:SOIC-8-1EP_3.9x4.9mm_P1.27mm_EP2.29x3mm -> Package_SO:SO-8_3.9x4.9mm_P1.27mm
Changed lines of the file:
@@
 F 0 "U6" H 2650 2450 50  0000 C CNN
 F 1 "IR2304" H 2650 2350 50  0000 C CNN
-F 2 "Package_SO:SOIC-8-1EP_3.9x4.9mm_P1.27mm_EP2.29x3mm" H 3050 1950 50  0001 C CIN
+F 2 "Package_SO:SO-8_3.9x4.9mm_P1.27mm" H 3050 1950 50  0001 C CIN
 F 3 "https://www.infineon.com/dgdl/ir2304.pdf?fileId=5546d462533600a4015355c9954a16e0" H 3050 1950 50  0001 C CNN
 	1    3050 1950
@@
 F 0 "U7" H 2600 4050 50  0000 C CNN
 F 1 "IR2304" H 2650 3950 50  0000 C CNN
-F 2 "Package_SO:SOIC-8-1EP_3.9x4.9mm_P1.27mm_EP2.29x3mm" H 3050 3650 50  0001 C CIN
+F 2 "Package_SO:SO-8_3.9x4.9mm_P1.27mm" H 3050 3650 50  0001 C CIN
 F 3 "https://www.infineon.com/dgdl/ir2304.pdf?fileId=5546d462533600a4015355c9954a16e0" H 3050 3650 50  0001 C CNN
 	1    3050 3650
@@
 F 0 "U8" H 2650 5700 50  0000 C CNN
 F 1 "IR2304" H 2650 5600 50  0000 C CNN
-F 2 "Package_SO:SOIC-8-1EP_3.9x4.9mm_P1.27mm_EP2.29x3mm" H 3050 5200 50  0001 C CIN
+F 2 "Package_SO:SO-8_3.9x4.9mm_P1.27mm" H 3050 5200 50  0001 C CIN
 F 3 "https://www.infineon.com/dgdl/ir2304.pdf?fileId=5546d462533600a4015355c9954a16e0" H 3050 5200 50  0001 C CNN
 	1    3050 5200
@@
 F 0 "R27" H 8120 2746 50  0000 L CNN
 F 1 "0R05" H 8120 2655 50  0000 L CNN
-F 2 "Resistor_SMD:R_2512_6332Metric" V 7980 2700 50  0001 C CNN
+F 2 "Resistor_SMD:R_4020_10251Metric_Pad1.65x5.30mm_HandSolder" V 7980 2700 50  0001 C CNN
 F 3 "~" H 8050 2700 50  0001 C CNN
 	1    8050 2700

Commit message: 29.08.20
Parts:
- added H3, H4, H6: MountingHole_Pad, user_pads:MountingHole_6x2, symbol Mechanical:MountingHole_Pad
- C12: footprint Capacitor_SMD:C_Elec_8x6.2 -> Capacitor_SMD:C_1206_3216Metric
Connections:
- net PA: now also H3.1
- net PB: now also H4.1
- net PC: now also H6.1
Changed lines of the file:
@@
 F 0 "C12" H 1568 6746 50  0000 L CNN
 F 1 "47 uF 35V" H 1568 6655 50  0000 L CNN
-F 2 "Capacitor_SMD:C_Elec_8x6.2" H 1488 6550 50  0001 C CNN
+F 2 "Capacitor_SMD:C_1206_3216Metric" H 1488 6550 50  0001 C CNN
 F 3 "~" H 1450 6700 50  0001 C CNN
 	1    1450 6700
@@
 	6500 3250 6500 2950
 Wire Wire Line
-	6500 3650 6500 4350
-Wire Wire Line
-	8050 3650 8050 4300
-Wire Wire Line
-	9450 3650 9450 4250
+	6500 3650 6500 4000
+Wire Wire Line
+	8050 3650 8050 4000
+Wire Wire Line
+	9450 3650 9450 4000
 $Comp
 L Transistor_FET:IRF540N Q7
@@
 Text Label 6950 5450 0    50   ~ 0
 Lock_S
+$Comp
+L Mechanical:MountingHole_Pad H3
+U 1 1 5F4CABDA
+P 6800 4000
+F 0 "H3" V 6754 4150 50  0000 L CNN
+F 1 "MountingHole_Pad" V 6845 4150 50  0000 L CNN
+F 2 "user_pads:MountingHole_6x2" H 6800 4000 50  0001 C CNN
+F 3 "~" H 6800 4000 50  0001 C CNN
+	1    6800 4000
+	0    1    1    0
+$EndComp
+$Comp
+L Mechanical:MountingHole_Pad H4
+U 1 1 5F4CB400
+P 8350 4000
+F 0 "H4" V 8304 4150 50  0000 L CNN
+F 1 "MountingHole_Pad" V 8395 4150 50  0000 L CNN
+F 2 "user_pads:MountingHole_6x2" H 8350 4000 50  0001 C CNN
+F 3 "~" H 8350 4000 50  0001 C CNN
+	1    8350 4000
+	0    1    1    0
+$EndComp
+$Comp
+L Mechanical:MountingHole_Pad H6
+U 1 1 5F4CC292
+P 9900 4000
+F 0 "H6" V 9854 4150 50  0000 L CNN
+F 1 "MountingHole_Pad" V 9945 4150 50  0000 L CNN
+F 2 "user_pads:MountingHole_6x2" H 9900 4000 50  0001 C CNN
+F 3 "~" H 9900 4000 50  0001 C CNN
+	1    9900 4000
+	0    1    1    0
+$EndComp
+Wire Wire Line
+	9800 4000 9450 4000
+Connection ~ 9450 4000
+Wire Wire Line
+	9450 4000 9450 4250
+Wire Wire Line
+	8250 4000 8050 4000
+Connection ~ 8050 4000
+Wire Wire Line
+	8050 4000 8050 4300
+Wire Wire Line
+	6700 4000 6500 4000
+Connection ~ 6500 4000
+Wire Wire Line
+	6500 4000 6500 4350
 $EndSCHEMATC

Commit message: --
Connections:
- net PA: now also H4.1; no longer H3.1
- net PB: now also H3.1; no longer H4.1
Other:
- moved on the sheet: H3, H4
Changed lines of the file:
@@
 	6500 3250 6500 2950
-Wire Wire Line
-	6500 3650 6500 4000
-Wire Wire Line
-	8050 3650 8050 4000
 Wire Wire Line
 	9450 3650 9450 4000
@@
 L Mechanical:MountingHole_Pad H3
 U 1 1 5F4CABDA
-P 6800 4000
-F 0 "H3" V 6754 4150 50  0000 L CNN
-F 1 "MountingHole_Pad" V 6845 4150 50  0000 L CNN
-F 2 "user_pads:MountingHole_6x2" H 6800 4000 50  0001 C CNN
-F 3 "~" H 6800 4000 50  0001 C CNN
-	1    6800 4000
+P 8200 4100
+F 0 "H3" V 8154 4250 50  0000 L CNN
+F 1 "MountingHole_Pad" V 8245 4250 50  0000 L CNN
+F 2 "user_pads:MountingHole_6x2" H 8200 4100 50  0001 C CNN
+F 3 "~" H 8200 4100 50  0001 C CNN
+	1    8200 4100
 	0    1    1    0
 $EndComp
@@
 L Mechanical:MountingHole_Pad H4
 U 1 1 5F4CB400
-P 8350 4000
-F 0 "H4" V 8304 4150 50  0000 L CNN
-F 1 "MountingHole_Pad" V 8395 4150 50  0000 L CNN
-F 2 "user_pads:MountingHole_6x2" H 8350 4000 50  0001 C CNN
-F 3 "~" H 8350 4000 50  0001 C CNN
-	1    8350 4000
+P 6700 4100
+F 0 "H4" V 6654 4250 50  0000 L CNN
+F 1 "MountingHole_Pad" V 6745 4250 50  0000 L CNN
+F 2 "user_pads:MountingHole_6x2" H 6700 4100 50  0001 C CNN
+F 3 "~" H 6700 4100 50  0001 C CNN
+	1    6700 4100
 	0    1    1    0
 $EndComp
@@
 	9450 4000 9450 4250
 Wire Wire Line
-	8250 4000 8050 4000
-Connection ~ 8050 4000
-Wire Wire Line
-	8050 4000 8050 4300
-Wire Wire Line
-	6700 4000 6500 4000
-Connection ~ 6500 4000
-Wire Wire Line
-	6500 4000 6500 4350
+	6500 3650 6500 4100
+Wire Wire Line
+	8050 3650 8050 4100
+Wire Wire Line
+	8100 4100 8050 4100
+Connection ~ 8050 4100
+Wire Wire Line
+	8050 4100 8050 4300
+Wire Wire Line
+	6600 4100 6500 4100
+Connection ~ 6500 4100
+Wire Wire Line
+	6500 4100 6500 4350
 $EndSCHEMATC
