File: shematic/bldc_drive/bldc_drive.sch (KiCad schematic (older format))
At the start: 0 parts

Commit message: 02.05.2020 01.18 --
Changed lines of the file:
@@
 $Descr A4 11693 8268
 encoding utf-8
-Sheet 1 3
+Sheet 1 4
 Title ""
 Date ""
@@
 Text Notes 1600 2750 0    394  ~ 0
 This project created for make\nBLCD motor controller
+$Sheet
+S 12550 3450 1200 650
+U 5EB1ABF5
+F0 "interfaces" 50
+F1 "interfaces.sch" 50
+$EndSheet
 $EndSCHEMATC

Commit message: 22.05.2020 21.40 --
Changed lines of the file:
@@
 $Descr A4 11693 8268
 encoding utf-8
-Sheet 1 4
+Sheet 1 5
 Title ""
 Date ""
@@
 F1 "interfaces.sch" 50
 $EndSheet
+$Sheet
+S 12550 4650 1200 500
+U 5ED063DC
+F0 "io_sheet" 50
+F1 "io_sheet.sch" 50
+$EndSheet
 $EndSCHEMATC

Commit message: 03.06.2020 21.40 --
Changed lines of the file:
@@
 $Descr A4 11693 8268
 encoding utf-8
-Sheet 1 5
+Sheet 1 6
 Title ""
 Date ""
@@
 F1 "io_sheet.sch" 50
 $EndSheet
+$Sheet
+S 12550 5600 1200 500
+U 5EDC2C23
+F0 "power_conv" 50
+F1 "power_conv.sch" 50
+$EndSheet
 $EndSCHEMATC
