File: shematic/bldc_drive/_autosave-FET_drive.sch (KiCad schematic (older format))
At the start: 51 parts, among them Q1 BC817, Q2 BC807, Q3 IRF1407, Q4 IRF1407, Q5 IRF1407, Q6 IRF1407, Q7 IRF1407, Q8 IRF1407, Q9 IRF1407, U6 IR2304, U7 IR2304, U8 IR2304, U9 INA193

Commit message: --
Parts:
- R23: footprint Resistor_SMD:R_0805_2012Metric -> Resistor_SMD:R_0603_1608Metric
Changed lines of the file:
@@
 F 0 "R23" V 6143 1750 50  0000 C CNN
 F 1 "1k" V 6234 1750 50  0000 C CNN
-F 2 "Resistor_SMD:R_0805_2012Metric" V 6280 1750 50  0001 C CNN
+F 2 "Resistor_SMD:R_0603_1608Metric" V 6280 1750 50  0001 C CNN
 F 3 "~" H 6350 1750 50  0001 C CNN
 	1    6350 1750
