File: shematic/bldc_drive/cpu_io.sch (KiCad schematic (older format))
At the start: 1 part

Commit message: 02.05.2020 01.18 --
Parts:
- added C?: 100n, symbol Device:C
- added C? (x4): 1u, symbol Device:C
- added D?: 1N4148WS, Diode_SMD:D_SOD-323, symbol Diode:1N4148WS
- added R?: 10k, symbol Device:R
Connections:
- net Vbat: now reaches U?.1 (VBAT)
- net Vbat: now also D?.1 (K)
- net GND: now reaches U?.23 (VSS)
- net GND: now also U?.35 (VSS), U?.47 (VSS), U?.8 (VSSA), C?.1, C?.1, C?.1, C?.1, C?.1
- net +3V3: now reaches U?.24 (VDD)
- net +3V3: now also U?.36 (VDDIO2), U?.48 (VDD), U?.9 (VDDA), C?.2, C?.2, C?.2, C?.2, D?.2 (A), R?.1
- net LAL: now reaches U?.26 (PB13)
- net LBL: now reaches U?.27 (PB14)
- net LCL: now reaches U?.28 (PB15)
- net LAH: now reaches U?.29 (PA8)
- net LBH: now reaches U?.30 (PA9)
- net LCH: now reaches U?.31 (PA10)
- net nRST: now reaches U?.7 (NRST)
- net nRST: now also C?.2, R?.2
Other:
- moved on the sheet: U?

Commit message: 10.05.2020 21.40 --
Parts:
- added C?: 1u, symbol Device:C
- added C? (x2): 15p, symbol Device:C
- added R? (x5): R, symbol Device:R
- added R?: 10k, symbol Device:R
- added U? (x3): A1302KUA-T, symbol Sensor_Magnetic:A1302KUA-T
- added U?: 24LC08, symbol Memory_EEPROM:24LC08
- added Y?: Crystal, symbol Device:Crystal
Connections:
- net labels added: +12V, BOOT0, CAN_RX, CAN_S, CAN_TX, CURRENT_SENSE, E_WP, HAL_A, HAL_B, HAL_C, RS485_DIR, RS485_RX, RS485_TX, SCL, SDA, U2RX, U2TX, V_POW_MEAS, Vin, Vin_ref, XT_IN, XT_OUT
- wire segments 27 -> 95

Commit message: 22.05.2020 21.40 --
Parts:
- added J1: Conn_01x04_Male, symbol Connector:Conn_01x04_Male
- gave numbers to parts that had none: 22
Connections:
- net labels added: DISC_IN_1, DISC_IN_2, LOCK_H, OD_OUT_1_MCU, SWDCLK, SWDIO, V_ANALOG_IO
- wire segments 95 -> 120
- no-connect marks 0 -> 2
Other:
- moved on the sheet: D1

Commit message: 11.06.2020 21.40 --
Parts:
- C1, C3, C6: footprint (none) -> Capacitor_SMD:C_0603_1608Metric
- C2, C4, C5, C7, C8: footprint (none) -> Capacitor_SMD:C_0805_2012Metric
- D1: footprint Diode_SMD:D_SOD-323 -> Diode_SMD:D_SOD-123
- J1: footprint (none) -> Connector_PinHeader_2.54mm:PinHeader_1x04_P2.54mm_Vertical
- R1, R2, R3, R4, R5, R6, R7: footprint (none) -> Resistor_SMD:R_0603_1608Metric
- U1: footprint (none) -> Package_SO:SO-8_3.9x4.9mm_P1.27mm
- U3, U4, U5: footprint (none) -> Package_SIP:SIP3_11.6x8.5mm
- Y1: footprint (none) -> Crystal:Crystal_HC49-4H_Vertical
Changed lines of the file:
@@
 F 0 "D1" V 5100 2150 50  0000 R CNN
 F 1 "1N4148WS" V 5000 2200 50  0000 R CNN
-F 2 "Diode_SMD:D_SOD-323" H 4950 1525 50  0001 C CNN
+F 2 "Diode_SMD:D_SOD-123" H 4950 1525 50  0001 C CNN
 F 3 "https://www.vishay.com/docs/85751/1n4148ws.pdf" H 4950 1700 50  0001 C CNN
 	1    4950 1700
@@
 F 0 "C1" H 1735 6854 50  0000 R CNN
 F 1 "100n" H 1735 6945 50  0000 R CNN
-F 2 "" H 1888 6750 50  0001 C CNN
+F 2 "Capacitor_SMD:C_0603_1608Metric" H 1888 6750 50  0001 C CNN
 F 3 "~" H 1850 6900 50  0001 C CNN
 	1    1850 6900
@@
 F 0 "R3" H 1920 6596 50  0000 L CNN
 F 1 "10k" H 1920 6505 50  0000 L CNN
-F 2 "" V 1780 6550 50  0001 C CNN
+F 2 "Resistor_SMD:R_0603_1608Metric" V 1780 6550 50  0001 C CNN
 F 3 "~" H 1850 6550 50  0001 C CNN
 	1    1850 6550
@@
 F 0 "C2" H 2285 6854 50  0000 R CNN
 F 1 "1u" H 2285 6945 50  0000 R CNN
-F 2 "" H 2438 6750 50  0001 C CNN
+F 2 "Capacitor_SMD:C_0805_2012Metric" H 2438 6750 50  0001 C CNN
 F 3 "~" H 2400 6900 50  0001 C CNN
 	1    2400 6900
@@
 F 0 "C4" H 2635 6854 50  0000 R CNN
 F 1 "1u" H 2635 6945 50  0000 R CNN
-F 2 "" H 2788 6750 50  0001 C CNN
+F 2 "Capacitor_SMD:C_0805_2012Metric" H 2788 6750 50  0001 C CNN
 F 3 "~" H 2750 6900 50  0001 C CNN
 	1    2750 6900
@@
 F 0 "C5" H 2985 6854 50  0000 R CNN
 F 1 "1u" H 2985 6945 50  0000 R CNN
-F 2 "" H 3138 6750 50  0001 C CNN
+F 2 "Capacitor_SMD:C_0805_2012Metric" H 3138 6750 50  0001 C CNN
 F 3 "~" H 3100 6900 50  0001 C CNN
 	1    3100 6900
@@
 F 0 "C7" H 3385 6854 50  0000 R CNN
 F 1 "1u" H 3385 6945 50  0000 R CNN
-F 2 "" H 3538 6750 50  0001 C CNN
+F 2 "Capacitor_SMD:C_0805_2012Metric" H 3538 6750 50  0001 C CNN
 F 3 "~" H 3500 6900 50  0001 C CNN
 	1    3500 6900
@@
 F 0 "U3" H 10420 1846 50  0000 R CNN
 F 1 "A1302KUA-T" H 10420 1755 50  0000 R CNN
-F 2 "" H 10650 1450 50  0001 L CIN
+F 2 "Package_SIP:SIP3_11.6x8.5mm" H 10650 1450 50  0001 L CIN
 F 3 "http://www.allegromicro.com/~/media/Files/Datasheets/A1301-2-Datasheet.ashx" H 10550 1800 50  0001 C CNN
 	1    10650 1800
@@
 F 0 "U4" H 10420 3346 50  0000 R CNN
 F 1 "A1302KUA-T" H 10420 3255 50  0000 R CNN
-F 2 "" H 10650 2950 50  0001 L CIN
+F 2 "Package_SIP:SIP3_11.6x8.5mm" H 10650 2950 50  0001 L CIN
 F 3 "http://www.allegromicro.com/~/media/Files/Datasheets/A1301-2-Datasheet.ashx" H 10550 3300 50  0001 C CNN
 	1    10650 3300
@@
 F 0 "U5" H 10420 4796 50  0000 R CNN
 F 1 "A1302KUA-T" H 10420 4705 50  0000 R CNN
-F 2 "" H 10650 4400 50  0001 L CIN
+F 2 "Package_SIP:SIP3_11.6x8.5mm" H 10650 4400 50  0001 L CIN
 F 3 "http://www.allegromicro.com/~/media/Files/Datasheets/A1301-2-Datasheet.ashx" H 10550 4750 50  0001 C CNN
 	1    10650 4750
@@
 F 0 "R6" H 10320 3096 50  0000 L CNN
 F 1 "R" H 10320 3005 50  0000 L CNN
-F 2 "" V 10180 3050 50  0001 C CNN
+F 2 "Resistor_SMD:R_0603_1608Metric" V 10180 3050 50  0001 C CNN
 F 3 "~" H 10250 3050 50  0001 C CNN
 	1    10250 3050
@@
 F 0 "R7" H 10320 4546 50  0000 L CNN
 F 1 "R" H 10320 4455 50  0000 L CNN
-F 2 "" V 10180 4500 50  0001 C CNN
+F 2 "Resistor_SMD:R_0603_1608Metric" V 10180 4500 50  0001 C CNN
 F 3 "~" H 10250 4500 50  0001 C CNN
 	1    10250 4500
@@
 F 0 "R5" H 10320 1596 50  0000 L CNN
 F 1 "R" H 10320 1505 50  0000 L CNN
-F 2 "" V 10180 1550 50  0001 C CNN
+F 2 "Resistor_SMD:R_0603_1608Metric" V 10180 1550 50  0001 C CNN
 F 3 "~" H 10250 1550 50  0001 C CNN
 	1    10250 1550
@@
 F 0 "U1" H 1450 4100 50  0000 C CNN
 F 1 "24LC08" H 1450 4000 50  0000 C CNN
-F 2 "" H 1750 3650 50  0001 C CNN
+F 2 "Package_SO:SO-8_3.9x4.9mm_P1.27mm" H 1750 3650 50  0001 C CNN
 F 3 "http://ww1.microchip.com/downloads/en/DeviceDoc/21710J.pdf" H 1750 3650 50  0001 C CNN
 	1    1750 3650
@@
 F 0 "C8" H 3885 6854 50  0000 R CNN
 F 1 "1u" H 3885 6945 50  0000 R CNN
-F 2 "" H 4038 6750 50  0001 C CNN
+F 2 "Capacitor_SMD:C_0805_2012Metric" H 4038 6750 50  0001 C CNN
 F 3 "~" H 4000 6900 50  0001 C CNN
 	1    4000 6900
@@
 F 0 "R1" H 1280 1254 50  0000 R CNN
 F 1 "R" H 1280 1345 50  0000 R CNN
-F 2 "" V 1280 1300 50  0001 C CNN
+F 2 "Resistor_SMD:R_0603_1608Metric" V 1280 1300 50  0001 C CNN
 F 3 "~" H 1350 1300 50  0001 C CNN
 	1    1350 1300
@@
 F 0 "R2" H 1280 1554 50  0000 R CNN
 F 1 "R" H 1280 1645 50  0000 R CNN
-F 2 "" V 1280 1600 50  0001 C CNN
+F 2 "Resistor_SMD:R_0603_1608Metric" V 1280 1600 50  0001 C CNN
 F 3 "~" H 1350 1600 50  0001 C CNN
 	1    1350 1600
@@
 F 0 "Y1" H 2850 1568 50  0000 C CNN
 F 1 "Crystal" H 2850 1477 50  0000 C CNN
-F 2 "" H 2850 1300 50  0001 C CNN
+F 2 "Crystal:Crystal_HC49-4H_Vertical" H 2850 1300 50  0001 C CNN
 F 3 "~" H 2850 1300 50  0001 C CNN
 	1    2850 1300
@@
 F 0 "C3" H 2385 1404 50  0000 R CNN
 F 1 "15p" H 2385 1495 50  0000 R CNN
-F 2 "" H 2538 1300 50  0001 C CNN
+F 2 "Capacitor_SMD:C_0603_1608Metric" H 2538 1300 50  0001 C CNN
 F 3 "~" H 2500 1450 50  0001 C CNN
 	1    2500 1450
@@
 F 0 "C6" H 3085 1404 50  0000 R CNN
 F 1 "15p" H 3085 1495 50  0000 R CNN
-F 2 "" H 3238 1300 50  0001 C CNN
+F 2 "Capacitor_SMD:C_0603_1608Metric" H 3238 1300 50  0001 C CNN
 F 3 "~" H 3200 1450 50  0001 C CNN
 	1    3200 1450
@@
 F 0 "R4" V 1743 3300 50  0000 C CNN
 F 1 "10k" V 1834 3300 50  0000 C CNN
-F 2 "" V 1880 3300 50  0001 C CNN
+F 2 "Resistor_SMD:R_0603_1608Metric" V 1880 3300 50  0001 C CNN
 F 3 "~" H 1950 3300 50  0001 C CNN
 	1    1950 3300
@@
 F 0 "J1" H 7822 1282 50  0000 R CNN
 F 1 "Conn_01x04_Male" H 7822 1373 50  0000 R CNN
-F 2 "" H 7850 1400 50  0001 C CNN
+F 2 "Connector_PinHeader_2.54mm:PinHeader_1x04_P2.54mm_Vertical" H 7850 1400 50  0001 C CNN
 F 3 "~" H 7850 1400 50  0001 C CNN
 	1    7850 1400

Commit message: --
Parts:
- U3, U4, U5: footprint Package_SIP:SIP3_11.6x8.5mm -> Package_TO_SOT_THT:TO-92_Wide
Changed lines of the file:
@@
 F 0 "U3" H 10420 1846 50  0000 R CNN
 F 1 "A1302KUA-T" H 10420 1755 50  0000 R CNN
-F 2 "Package_SIP:SIP3_11.6x8.5mm" H 10650 1450 50  0001 L CIN
+F 2 "Package_TO_SOT_THT:TO-92_Wide" H 10650 1450 50  0001 L CIN
 F 3 "http://www.allegromicro.com/~/media/Files/Datasheets/A1301-2-Datasheet.ashx" H 10550 1800 50  0001 C CNN
 	1    10650 1800
@@
 F 0 "U4" H 10420 3346 50  0000 R CNN
 F 1 "A1302KUA-T" H 10420 3255 50  0000 R CNN
-F 2 "Package_SIP:SIP3_11.6x8.5mm" H 10650 2950 50  0001 L CIN
+F 2 "Package_TO_SOT_THT:TO-92_Wide" H 10650 2950 50  0001 L CIN
 F 3 "http://www.allegromicro.com/~/media/Files/Datasheets/A1301-2-Datasheet.ashx" H 10550 3300 50  0001 C CNN
 	1    10650 3300
@@
 F 0 "U5" H 10420 4796 50  0000 R CNN
 F 1 "A1302KUA-T" H 10420 4705 50  0000 R CNN
-F 2 "Package_SIP:SIP3_11.6x8.5mm" H 10650 4400 50  0001 L CIN
+F 2 "Package_TO_SOT_THT:TO-92_Wide" H 10650 4400 50  0001 L CIN
 F 3 "http://www.allegromicro.com/~/media/Files/Datasheets/A1301-2-Datasheet.ashx" H 10550 4750 50  0001 C CNN
 	1    10650 4750

Commit message: 29.08.20
Parts:
- removed C3, C6: 15p, Capacitor_SMD:C_0603_1608Metric, symbol Device:C
- removed Y1: Crystal, Crystal:Crystal_HC49-4H_Vertical, symbol Device:Crystal
- added R38, R43: 10k, Resistor_SMD:R_0603_1608Metric, symbol Device:R
- added Y2: Crystal_GND2_Small, Crystal:Resonator_SMD_muRata_CSTxExxV-3Pin_3.0x1.1mm, symbol Device:Crystal_GND2_Small
- J1: footprint Connector_PinHeader_2.54mm:PinHeader_1x04_P2.54mm_Vertical -> Connector_PinHeader_1.00mm:PinHeader_1x04_P1.00mm_Vertical
Connections:
- net +3V3: now also R38.1, R43.1
- net GND: now also Y2.2
- net SCL: now also R38.2
- net SDA: now also R43.2
- net XT_IN: now also Y2.1
- net XT_OUT: now also Y2.3
Changed lines of the file:
@@
 L power:+3V3 #PWR0128
 U 1 1 5EC1D29F
-P 1750 3250
-F 0 "#PWR0128" H 1750 3100 50  0001 C CNN
-F 1 "+3V3" H 1765 3423 50  0000 C CNN
-F 2 "" H 1750 3250 50  0001 C CNN
-F 3 "" H 1750 3250 50  0001 C CNN
-	1    1750 3250
+P 1750 2650
+F 0 "#PWR0128" H 1750 2500 50  0001 C CNN
+F 1 "+3V3" H 1765 2823 50  0000 C CNN
+F 2 "" H 1750 2650 50  0001 C CNN
+F 3 "" H 1750 2650 50  0001 C CNN
+	1    1750 2650
 	1    0    0    -1
 $EndComp
@@
 	1750 4000 1750 4050
 Wire Wire Line
-	2150 3550 2350 3550
-Wire Wire Line
-	2150 3650 2350 3650
+	2150 3650 2250 3650
 Text Label 2350 3550 0    50   ~ 0
 SDA
@@
 BOOT0
 $Comp
-L Device:Crystal Y1
-U 1 1 5EC44465
-P 2850 1300
-F 0 "Y1" H 2850 1568 50  0000 C CNN
-F 1 "Crystal" H 2850 1477 50  0000 C CNN
-F 2 "Crystal:Crystal_HC49-4H_Vertical" H 2850 1300 50  0001 C CNN
-F 3 "~" H 2850 1300 50  0001 C CNN
-	1    2850 1300
-	1    0    0    -1
-$EndComp
-$Comp
-L Device:C C3
-U 1 1 5EC477DC
-P 2500 1450
-F 0 "C3" H 2385 1404 50  0000 R CNN
-F 1 "15p" H 2385 1495 50  0000 R CNN
-F 2 "Capacitor_SMD:C_0603_1608Metric" H 2538 1300 50  0001 C CNN
-F 3 "~" H 2500 1450 50  0001 C CNN
-	1    2500 1450
-	-1   0    0    1
-$EndComp
-$Comp
-L Device:C C6
-U 1 1 5EC49099
-P 3200 1450
-F 0 "C6" H 3085 1404 50  0000 R CNN
-F 1 "15p" H 3085 1495 50  0000 R CNN
-F 2 "Capacitor_SMD:C_0603_1608Metric" H 3238 1300 50  0001 C CNN
-F 3 "~" H 3200 1450 50  0001 C CNN
-	1    3200 1450
-	-1   0    0    1
-$EndComp
-Wire Wire Line
-	2700 1300 2500 1300
-Wire Wire Line
-	3000 1300 3200 1300
-$Comp
 L power:GND #PWR0133
 U 1 1 5EC4DABE
@@
 $EndComp
 Wire Wire Line
-	2500 1600 2850 1600
-Wire Wire Line
-	2850 1650 2850 1600
-Connection ~ 2850 1600
-Wire Wire Line
-	2850 1600 3200 1600
-Wire Wire Line
-	3200 1300 3400 1300
-Connection ~ 3200 1300
-Text Label 3400 1300 2    50   ~ 0
-XT_IN
-Wire Wire Line
-	2500 1300 2300 1300
-Connection ~ 2500 1300
-Text Label 2300 1300 0    50   ~ 0
-XT_OUT
-Wire Wire Line
 	4550 2350 3900 2350
 Wire Wire Line
@@
 Connection ~ 1750 3300
 Wire Wire Line
-	1750 3300 1750 3250
-Wire Wire Line
 	2100 3300 2200 3300
-Wire Wire Line
-	2200 3300 2200 3750
 Connection ~ 2200 3750
 Wire Wire Line
@@
 F 0 "J1" H 7822 1282 50  0000 R CNN
 F 1 "Conn_01x04_Male" H 7822 1373 50  0000 R CNN
-F 2 "Connector_PinHeader_2.54mm:PinHeader_1x04_P2.54mm_Vertical" H 7850 1400 50  0001 C CNN
+F 2 "Connector_PinHeader_1.00mm:PinHeader_1x04_P1.00mm_Vertical" H 7850 1400 50  0001 C CNN
 F 3 "~" H 7850 1400 50  0001 C CNN
 	1    7850 1400
@@
 Text GLabel 3850 4350 0    50   Input ~ 0
 LOCK_H
+$Comp
+L Device:R R43
+U 1 1 5F5B00ED
+P 1950 3000
+F 0 "R43" V 1743 3000 50  0000 C CNN
+F 1 "10k" V 1834 3000 50  0000 C CNN
+F 2 "Resistor_SMD:R_0603_1608Metric" V 1880 3000 50  0001 C CNN
+F 3 "~" H 1950 3000 50  0001 C CNN
+	1    1950 3000
+	0    -1   1    0
+$EndComp
+$Comp
+L Device:R R38
+U 1 1 5F5B0607
+P 1950 2700
+F 0 "R38" V 1743 2700 50  0000 C CNN
+F 1 "10k" V 1834 2700 50  0000 C CNN
+F 2 "Resistor_SMD:R_0603_1608Metric" V 1880 2700 50  0001 C CNN
+F 3 "~" H 1950 2700 50  0001 C CNN
+	1    1950 2700
+	0    -1   1    0
+$EndComp
+Wire Wire Line
+	2200 3300 2200 3750
+Wire Wire Line
+	2150 3550 2350 3550
+Wire Wire Line
+	2100 3000 2150 3000
+Wire Wire Line
+	2150 3000 2150 3550
+Connection ~ 2150 3550
+Wire Wire Line
+	2100 2700 2250 2700
+Wire Wire Line
+	2250 2700 2250 3650
+Connection ~ 2250 3650
+Wire Wire Line
+	2250 3650 2350 3650
+Wire Wire Line
+	1800 2700 1750 2700
+Wire Wire Line
+	1750 2700 1750 2650
+Wire Wire Line
+	1750 2700 1750 3000
+Connection ~ 1750 2700
+Wire Wire Line
+	1800 3000 1750 3000
+Connection ~ 1750 3000
+Wire Wire Line
+	1750 3000 1750 3300
+$Comp
+L Device:Crystal_GND2_Small Y2
+U 1 1 5F5DD1F0
+P 2850 1400
+F 0 "Y2" H 2850 1625 50  0000 C CNN
+F 1 "Crystal_GND2_Small" H 2850 1534 50  0000 C CNN
+F 2 "Crystal:Resonator_SMD_muRata_CSTxExxV-3Pin_3.0x1.1mm" H 2850 1400 50  0001 C CNN
+F 3 "~" H 2850 1400 50  0001 C CNN
+	1    2850 1400
+	1    0    0    -1
+$EndComp
+Wire Wire Line
+	2850 1500 2850 1650
+Wire Wire Line
+	2950 1400 3200 1400
+Wire Wire Line
+	2750 1400 2500 1400
+Text Label 3200 1400 0    50   ~ 0
+XT_OUT
+Text Label 2500 1400 2    50   ~ 0
+XT_IN
 $EndSCHEMATC

Commit message: --
Parts:
- C2: footprint Capacitor_SMD:C_0805_2012Metric -> Capacitor_SMD:C_0603_1608Metric
- C3: renamed from C4; footprint Capacitor_SMD:C_0805_2012Metric -> Capacitor_SMD:C_0603_1608Metric
- C4: renamed from C5; footprint Capacitor_SMD:C_0805_2012Metric -> Capacitor_SMD:C_0603_1608Metric
- C5: renamed from C7; footprint Capacitor_SMD:C_0805_2012Metric -> Capacitor_SMD:C_0603_1608Metric
- C6: renamed from C8; footprint Capacitor_SMD:C_0805_2012Metric -> Capacitor_SMD:C_0603_1608Metric
- renumbered R38 to R4, R43 to R5, R4 to R6, R5 to R7, R6 to R8, R7 to R9, Y2 to Y1
