File: shematic/bldc_drive/cpu_io.sch (KiCad schematic (older format))
At the start: 23 parts, among them J1 Conn_01x04_Male, U1 24LC08, U2 STM32F042C6Tx, U3 A1302KUA-T, U4 A1302KUA-T, U5 A1302KUA-T, Y1 Crystal_GND2_Small

Commit message: --
Parts:
- U1: footprint Package_SO:SO-8_3.9x4.9mm_P1.27mm -> Package_SO:SOIC-8_3.9x4.9mm_P1.27mm
Changed lines of the file:
@@
 F 0 "U1" H 1450 4100 50  0000 C CNN
 F 1 "24LC08" H 1450 4000 50  0000 C CNN
-F 2 "Package_SO:SO-8_3.9x4.9mm_P1.27mm" H 1750 3650 50  0001 C CNN
+F 2 "Package_SO:SOIC-8_3.9x4.9mm_P1.27mm" H 1750 3650 50  0001 C CNN
 F 3 "http://ww1.microchip.com/downloads/en/DeviceDoc/21710J.pdf" H 1750 3650 50  0001 C CNN
 	1    1750 3650
