File: shematic/bldc_drive/interfaces.sch (KiCad schematic (older format))
At the start: 15 parts

Commit message: 10.05.2020 21.40 --
Parts:
- added C? (x2): 1u, symbol Device:C
- added D? (x2): DZ2S033X0L, Diode_SMD:D_SOD-523, symbol Diode:DZ2S033X0L
- R? (x2): value 120R -> 4k7
- R? (x2): value 120R -> 2k2
Connections:
- wire segments 61 -> 88
Other:
- moved on the sheet: J?
Changed lines of the file:
@@
 ext_RX
 Wire Wire Line
-	4000 4900 4100 4900
+	4000 4900 4050 4900
 Text GLabel 3000 4900 0    50   Input ~ 0
 U2TX
@@
 U 1 1 5EB1D336
 P 3600 6200
-F 0 "U?" H 3200 6600 50  0000 L CNN
-F 1 "SN74AUP1T34DCK" H 2650 6500 50  0000 L CNN
+F 0 "U?" H 3250 5900 50  0000 L CNN
+F 1 "SN74AUP1T34DCK" H 2650 5750 50  0000 L CNN
 F 2 "Package_TO_SOT_SMD:SOT-353_SC-70-5" H 3600 5500 50  0001 C CNN
 F 3 "http://www.ti.com/lit/ds/symlink/sn74aup1t34.pdf" H 3600 5600 50  0001 C CNN
@@
 $EndComp
 Wire Wire Line
-	3700 5900 3700 5600
+	3700 5900 3700 5750
 Wire Wire Line
 	3500 5900 3500 5750
 Wire Wire Line
-	4000 6200 4100 6200
+	4000 6200 4050 6200
 Wire Wire Line
 	3600 6550 3600 6500
@@
 L Connector:Conn_01x04_Male J?
 U 1 1 5EB43A6E
-P 4800 5600
-F 0 "J?" H 4908 5881 50  0000 C CNN
-F 1 "Conn_01x04_Male" H 4908 5790 50  0000 C CNN
-F 2 "" H 4800 5600 50  0001 C CNN
-F 3 "~" H 4800 5600 50  0001 C CNN
-	1    4800 5600
-	1    0    0    -1
+P 4550 5450
+F 0 "J?" H 4500 5800 50  0000 C CNN
+F 1 "Conn_01x04_Male" H 4250 5700 50  0000 C CNN
+F 2 "" H 4550 5450 50  0001 C CNN
+F 3 "~" H 4550 5450 50  0001 C CNN
+	1    4550 5450
+	-1   0    0    -1
 $EndComp
 $Comp
 L Connector:Conn_01x04_Male J?
 U 1 1 5EB44CD9
-P 9200 3600
-F 0 "J?" H 9308 3881 50  0000 C CNN
-F 1 "Conn_01x04_Male" H 9308 3790 50  0000 C CNN
-F 2 "" H 9200 3600 50  0001 C CNN
-F 3 "~" H 9200 3600 50  0001 C CNN
-	1    9200 3600
+P 8700 3600
+F 0 "J?" H 8808 3881 50  0000 C CNN
+F 1 "Conn_01x04_Male" H 8808 3790 50  0000 C CNN
+F 2 "" H 8700 3600 50  0001 C CNN
+F 3 "~" H 8700 3600 50  0001 C CNN
+	1    8700 3600
 	-1   0    0    -1
 $EndComp
@@
 P 8200 4200
 F 0 "R?" H 8130 4154 50  0000 R CNN
-F 1 "120R" H 8130 4245 50  0000 R CNN
+F 1 "4k7" H 8130 4245 50  0000 R CNN
 F 2 "" V 8130 4200 50  0001 C CNN
 F 3 "~" H 8200 4200 50  0001 C CNN
@@
 P 8200 4650
 F 0 "R?" H 8130 4604 50  0000 R CNN
-F 1 "120R" H 8130 4695 50  0000 R CNN
+F 1 "2k2" H 8130 4695 50  0000 R CNN
 F 2 "" V 8130 4650 50  0001 C CNN
 F 3 "~" H 8200 4650 50  0001 C CNN
@@
 P 7850 4200
 F 0 "R?" H 7780 4154 50  0000 R CNN
-F 1 "120R" H 7780 4245 50  0000 R CNN
+F 1 "4k7" H 7780 4245 50  0000 R CNN
 F 2 "" V 7780 4200 50  0001 C CNN
 F 3 "~" H 7850 4200 50  0001 C CNN
@@
 P 7850 4650
 F 0 "R?" H 7780 4604 50  0000 R CNN
-F 1 "120R" H 7780 4695 50  0000 R CNN
+F 1 "2k2" H 7780 4695 50  0000 R CNN
 F 2 "" V 7780 4650 50  0001 C CNN
 F 3 "~" H 7850 4650 50  0001 C CNN
@@
 Wire Wire Line
 	7850 4500 7850 4350
-Wire Wire Line
-	7850 4050 7850 3950
 $Comp
 L power:+12V #PWR?
 U 1 1 5EB4D68E
-P 7850 3850
-F 0 "#PWR?" H 7850 3700 50  0001 C CNN
-F 1 "+12V" H 7865 4023 50  0000 C CNN
-F 2 "" H 7850 3850 50  0001 C CNN
-F 3 "" H 7850 3850 50  0001 C CNN
-	1    7850 3850
+P 7850 3250
+F 0 "#PWR?" H 7850 3100 50  0001 C CNN
+F 1 "+12V" H 7865 3423 50  0000 C CNN
+F 2 "" H 7850 3250 50  0001 C CNN
+F 3 "" H 7850 3250 50  0001 C CNN
+	1    7850 3250
 	1    0    0    -1
 $EndComp
@@
 	8200 4050 8200 3500
 Wire Wire Line
-	8200 3500 9000 3500
-Wire Wire Line
-	9000 3800 9000 5050
-Wire Wire Line
-	9000 5050 8200 5050
+	8200 3500 8500 3500
 Connection ~ 8200 5050
-Wire Wire Line
-	9000 3700 8100 3700
-Wire Wire Line
-	8100 3700 8100 3950
-Wire Wire Line
-	8100 3950 7850 3950
-Connection ~ 7850 3950
-Wire Wire Line
-	7850 3950 7850 3850
-Text GLabel 7050 4350 0    50   Input ~ 0
+Text GLabel 6550 4350 0    50   Input ~ 0
 Vin_ref
-Text GLabel 7050 4450 0    50   Input ~ 0
+Text GLabel 6550 4450 0    50   Input ~ 0
 Vin
-Wire Wire Line
-	7050 4450 8200 4450
 Connection ~ 8200 4450
 Wire Wire Line
 	8200 4450 8200 4350
-Wire Wire Line
-	7050 4350 7850 4350
 Connection ~ 7850 4350
+$Comp
+L power:GND #PWR?
+U 1 1 5EB84885
+P 8200 5150
+F 0 "#PWR?" H 8200 4900 50  0001 C CNN
+F 1 "GND" H 8205 4977 50  0000 C CNN
+F 2 "" H 8200 5150 50  0001 C CNN
+F 3 "" H 8200 5150 50  0001 C CNN
+	1    8200 5150
+	1    0    0    -1
+$EndComp
+Wire Wire Line
+	8200 5150 8200 5050
+Wire Wire Line
+	7850 4050 7850 3700
+Connection ~ 7850 3700
+Wire Wire Line
+	7850 3700 7850 3250
+Wire Wire Line
+	7850 3700 8500 3700
+Wire Wire Line
+	8500 3800 8500 5050
+Wire Wire Line
+	8500 5050 8200 5050
+$Comp
+L power:GND #PWR?
+U 1 1 5EB902FC
+P 4300 5700
+F 0 "#PWR?" H 4300 5450 50  0001 C CNN
+F 1 "GND" H 4305 5527 50  0000 C CNN
+F 2 "" H 4300 5700 50  0001 C CNN
+F 3 "" H 4300 5700 50  0001 C CNN
+	1    4300 5700
+	1    0    0    -1
+$EndComp
+Wire Wire Line
+	4050 5350 4050 4900
+Connection ~ 4050 4900
+Wire Wire Line
+	4050 4900 4100 4900
+Wire Wire Line
+	4050 5450 4050 6200
+Connection ~ 4050 6200
+Wire Wire Line
+	4050 6200 4100 6200
+Wire Wire Line
+	4350 5350 4050 5350
+Wire Wire Line
+	4350 5450 4050 5450
+Wire Wire Line
+	4300 5700 4300 5650
+Wire Wire Line
+	4300 5650 4350 5650
+Wire Wire Line
+	4350 5550 4150 5550
+Wire Wire Line
+	4150 5550 4150 5750
+Wire Wire Line
+	4150 5750 3700 5750
+Connection ~ 3700 5750
+Wire Wire Line
+	3700 5750 3700 5600
+$Comp
+L Diode:DZ2S033X0L D?
+U 1 1 5EB99258
+P 6750 4750
+F 0 "D?" V 6650 4600 50  0000 L CNN
+F 1 "DZ2S033X0L" V 7250 4600 50  0001 L CNN
+F 2 "Diode_SMD:D_SOD-523" H 6750 4575 50  0001 C CNN
+F 3 "https://industrial.panasonic.com/content/data/SC/ds/ds4/DZ2S03300L_E.pdf" H 6750 4750 50  0001 C CNN
+	1    6750 4750
+	0    1    1    0
+$EndComp
+$Comp
+L Diode:DZ2S033X0L D?
+U 1 1 5EB9B699
+P 7600 4750
+F 0 "D?" V 7500 4650 50  0000 L CNN
+F 1 "DZ2S033X0L" V 8100 4800 50  0001 L CNN
+F 2 "Diode_SMD:D_SOD-523" H 7600 4575 50  0001 C CNN
+F 3 "https://industrial.panasonic.com/content/data/SC/ds/ds4/DZ2S03300L_E.pdf" H 7600 4750 50  0001 C CNN
+	1    7600 4750
+	0    1    1    0
+$EndComp
+Wire Wire Line
+	7300 5050 7600 5050
+Connection ~ 7850 5050
+Wire Wire Line
+	7600 4900 7600 5050
+Connection ~ 7600 5050
+Wire Wire Line
+	7600 5050 7850 5050
+Wire Wire Line
+	7600 4600 7600 4450
+Connection ~ 7600 4450
+Wire Wire Line
+	7600 4450 8200 4450
+$Comp
+L Device:C C?
+U 1 1 5EBA30CC
+P 7300 4750
+F 0 "C?" H 7415 4796 50  0000 L CNN
+F 1 "1u" H 7415 4705 50  0000 L CNN
+F 2 "" H 7338 4600 50  0001 C CNN
+F 3 "~" H 7300 4750 50  0001 C CNN
+	1    7300 4750
+	1    0    0    -1
+$EndComp
+$Comp
+L Device:C C?
+U 1 1 5EBA4AA2
+P 6950 4750
+F 0 "C?" H 7065 4796 50  0000 L CNN
+F 1 "1u" H 7065 4705 50  0000 L CNN
+F 2 "" H 6988 4600 50  0001 C CNN
+F 3 "~" H 6950 4750 50  0001 C CNN
+	1    6950 4750
+	1    0    0    -1
+$EndComp
+Wire Wire Line
+	7300 4900 7300 5050
+Wire Wire Line
+	7300 4600 7300 4450
+Connection ~ 7300 4450
+Wire Wire Line
+	7300 4450 7600 4450
+Wire Wire Line
+	6550 4450 7300 4450
+Wire Wire Line
+	6550 4350 6750 4350
+Wire Wire Line
+	6750 4600 6750 4350
+Connection ~ 6750 4350
+Wire Wire Line
+	6750 4350 6950 4350
+Wire Wire Line
+	6950 4600 6950 4350
+Connection ~ 6950 4350
+Wire Wire Line
+	6950 4350 7850 4350
+Wire Wire Line
+	6750 4900 6750 5050
+Wire Wire Line
+	6750 5050 6950 5050
+Connection ~ 7300 5050
+Wire Wire Line
+	6950 4900 6950 5050
+Connection ~ 6950 5050
+Wire Wire Line
+	6950 5050 7300 5050
 $EndSCHEMATC

Commit message: 22.05.2020 21.40 --
Parts:
- removed C? (x2): 1u, symbol Device:C
- removed D? (x2): DZ2S033X0L, Diode_SMD:D_SOD-523, symbol Diode:DZ2S033X0L
- removed J?: Conn_01x04_Male, symbol Connector:Conn_01x04_Male
- removed R? (x2): 4k7, symbol Device:R
- removed R? (x2): 2k2, symbol Device:R
- gave numbers to parts that had none: 10
Connections:
- net labels removed: +12V, Vin, Vin_ref
- wire segments 88 -> 56
- no-connect marks 0 -> 4
Other:
- moved on the sheet: R32, R33, SW1

Commit message: 11.06.2020 21.40 --
Parts:
- removed SW1: SW_DIP_x04, symbol Switch:SW_DIP_x04
- added J4, J5: Conn_01x02_Male, Connector_PinHeader_2.54mm:PinHeader_1x02_P2.54mm_Vertical, symbol Connector:Conn_01x02_Male
- C14, C15: footprint (none) -> Capacitor_SMD:C_0805_2012Metric
- J2: footprint (none) -> Connector_PinHeader_2.54mm:PinHeader_1x04_P2.54mm_Vertical
- R32, R33: footprint (none) -> Resistor_SMD:R_1206_3216Metric
- U11: footprint (none) -> Package_SO:SOIC-8-1EP_3.9x4.9mm_P1.27mm_EP2.29x3mm
Connections:
- no-connect marks 4 -> 0
Other:
- note added: "CAN Term Resistor ON"
- note added: "RS485 Term Resistor ON"
- note removed: "SW1 CAN Term Resistor ON"
- note removed: "SW2 RS485 Term Resistor ON"
Changed lines of the file:
@@
 F 0 "U11" H 3800 3800 50  0000 C CNN
 F 1 "MAX481E" H 3900 3700 50  0000 C CNN
-F 2 "" H 3600 2500 50  0001 C CNN
+F 2 "Package_SO:SOIC-8-1EP_3.9x4.9mm_P1.27mm_EP2.29x3mm" H 3600 2500 50  0001 C CNN
 F 3 "https://datasheets.maximintegrated.com/en/ds/MAX1487E-MAX491E.pdf" H 3600 3250 50  0001 C CNN
 	1    3600 3200
@@
 F 0 "R32" V 5493 800 50  0000 C CNN
 F 1 "120R" V 5584 800 50  0000 C CNN
-F 2 "" V 5630 800 50  0001 C CNN
+F 2 "Resistor_SMD:R_1206_3216Metric" V 5630 800 50  0001 C CNN
 F 3 "~" H 5700 800 50  0001 C CNN
 	1    5700 800
@@
 Text Label 6250 800  0    50   ~ 0
 CAN_RES_SW
-Wire Wire Line
-	7450 950  7100 950
-Wire Wire Line
-	8050 950  8400 950
-Text Label 7100 950  0    50   ~ 0
-CAN_RES_SW
-Text Label 8150 950  0    50   ~ 0
-CAN_H
-Text Notes 8700 950  0    50   ~ 0
-SW1 CAN Term Resistor ON
+Text Notes 8050 1700 0    50   ~ 0
+ CAN Term Resistor ON
 Text GLabel 2850 1350 0    50   Input ~ 0
 CAN_TX
@@
 F 0 "R33" V 5593 1150 50  0000 C CNN
 F 1 "120R" V 5684 1150 50  0000 C CNN
-F 2 "" V 5730 1150 50  0001 C CNN
+F 2 "Resistor_SMD:R_1206_3216Metric" V 5730 1150 50  0001 C CNN
 F 3 "~" H 5800 1150 50  0001 C CNN
 	1    5800 1150
@@
 Text Label 6000 1150 0    50   ~ 0
 RS485_TERM
-Text Label 7000 1050 0    50   ~ 0
-RS485_TERM
-Wire Wire Line
-	7000 1050 7450 1050
-Wire Wire Line
-	8050 1050 8400 1050
-Text Label 8100 1050 0    50   ~ 0
-RS485_B
-Text Notes 8700 1050 0    50   ~ 0
-SW2 RS485 Term Resistor ON
+Text Notes 8050 2050 0    50   ~ 0
+ RS485 Term Resistor ON
 Text GLabel 2850 3100 0    50   Input ~ 0
 RS485_RX
@@
 F 0 "C15" H 2265 5496 50  0000 L CNN
 F 1 "1u" H 2265 5405 50  0000 L CNN
-F 2 "" H 2188 5300 50  0001 C CNN
+F 2 "Capacitor_SMD:C_0805_2012Metric" H 2188 5300 50  0001 C CNN
 F 3 "~" H 2150 5450 50  0001 C CNN
 	1    2150 5450
@@
 F 0 "C14" H 1915 5496 50  0000 L CNN
 F 1 "1u" H 1915 5405 50  0000 L CNN
-F 2 "" H 1838 5300 50  0001 C CNN
+F 2 "Capacitor_SMD:C_0805_2012Metric" H 1838 5300 50  0001 C CNN
 F 3 "~" H 1800 5450 50  0001 C CNN
 	1    1800 5450
@@
 F 0 "J2" H 4500 5800 50  0000 C CNN
 F 1 "Conn_01x04_Male" H 4250 5700 50  0000 C CNN
-F 2 "" H 4550 5450 50  0001 C CNN
+F 2 "Connector_PinHeader_2.54mm:PinHeader_1x04_P2.54mm_Vertical" H 4550 5450 50  0001 C CNN
 F 3 "~" H 4550 5450 50  0001 C CNN
 	1    4550 5450
@@
 	3700 5750 3700 5600
 $Comp
-L Switch:SW_DIP_x04 SW1
-U 1 1 5EB1EA3E
-P 7750 1150
-F 0 "SW1" H 7750 1617 50  0000 C CNN
-F 1 "SW_DIP_x04" H 7750 1526 50  0000 C CNN
-F 2 "" H 7750 1150 50  0001 C CNN
-F 3 "~" H 7750 1150 50  0001 C CNN
-	1    7750 1150
-	1    0    0    -1
-$EndComp
-NoConn ~ 8050 1150
-NoConn ~ 8050 1250
-NoConn ~ 7450 1150
-NoConn ~ 7450 1250
+L Connector:Conn_01x02_Male J4
+U 1 1 5EF64825
+P 7800 1650
+F 0 "J4" H 7908 1831 50  0000 C CNN
+F 1 "Conn_01x02_Male" H 7908 1740 50  0000 C CNN
+F 2 "Connector_PinHeader_2.54mm:PinHeader_1x02_P2.54mm_Vertical" H 7800 1650 50  0001 C CNN
+F 3 "~" H 7800 1650 50  0001 C CNN
+	1    7800 1650
+	-1   0    0    -1
+$EndComp
+$Comp
+L Connector:Conn_01x02_Male J5
+U 1 1 5EF65E29
+P 7800 1950
+F 0 "J5" H 7954 1762 50  0000 R CNN
+F 1 "Conn_01x02_Male" H 8150 1650 50  0000 R CNN
+F 2 "Connector_PinHeader_2.54mm:PinHeader_1x02_P2.54mm_Vertical" H 7800 1950 50  0001 C CNN
+F 3 "~" H 7800 1950 50  0001 C CNN
+	1    7800 1950
+	-1   0    0    -1
+$EndComp
+Wire Wire Line
+	7600 1650 7300 1650
+Wire Wire Line
+	7600 1750 7300 1750
+Text Label 7300 1650 2    50   ~ 0
+CAN_H
+Text Label 7300 1750 2    50   ~ 0
+CAN_RES_SW
+Text Label 7300 2050 2    50   ~ 0
+RS485_TERM
+Text Label 7300 1950 2    50   ~ 0
+RS485_B
+Wire Wire Line
+	7600 2050 7300 2050
+Wire Wire Line
+	7600 1950 7300 1950
 $EndSCHEMATC

Commit message: 29.08.20
Parts:
- J2: footprint Connector_PinHeader_2.54mm:PinHeader_1x04_P2.54mm_Vertical -> Connector_PinHeader_1.27mm:PinHeader_1x04_P1.27mm_Vertical
- U11: footprint Package_SO:SOIC-8-1EP_3.9x4.9mm_P1.27mm_EP2.29x3mm -> Package_SO:SOIC-8_3.9x4.9mm_P1.27mm
Connections:
- net CAN_H: now also R32.1
- net CAN_L: now also J4.2 (Pin_2)
- net RS485_A: now also J5.2 (Pin_2)
- net RS485_B: now also R33.1
- removed net CAN_RES_SW: J4.2 (Pin_2), R32.1
- removed net RS485_TERM: J5.2 (Pin_2), R33.1
Changed lines of the file:
@@
 F 0 "U11" H 3800 3800 50  0000 C CNN
 F 1 "MAX481E" H 3900 3700 50  0000 C CNN
-F 2 "Package_SO:SOIC-8-1EP_3.9x4.9mm_P1.27mm_EP2.29x3mm" H 3600 2500 50  0001 C CNN
+F 2 "Package_SO:SOIC-8_3.9x4.9mm_P1.27mm" H 3600 2500 50  0001 C CNN
 F 3 "https://datasheets.maximintegrated.com/en/ds/MAX1487E-MAX491E.pdf" H 3600 3250 50  0001 C CNN
 	1    3600 3200
@@
 Wire Wire Line
 	5300 800  5550 800
-Wire Wire Line
-	5850 800  6250 800
-Text Label 6250 800  0    50   ~ 0
-CAN_RES_SW
 Text Notes 8050 1700 0    50   ~ 0
  CAN Term Resistor ON
@@
 Text Label 5300 1150 0    50   ~ 0
 RS485_A
-Wire Wire Line
-	5950 1150 6400 1150
-Text Label 6000 1150 0    50   ~ 0
-RS485_TERM
 Text Notes 8050 2050 0    50   ~ 0
  RS485 Term Resistor ON
@@
 F 0 "J2" H 4500 5800 50  0000 C CNN
 F 1 "Conn_01x04_Male" H 4250 5700 50  0000 C CNN
-F 2 "Connector_PinHeader_2.54mm:PinHeader_1x04_P2.54mm_Vertical" H 4550 5450 50  0001 C CNN
+F 2 "Connector_PinHeader_1.27mm:PinHeader_1x04_P1.27mm_Vertical" H 4550 5450 50  0001 C CNN
 F 3 "~" H 4550 5450 50  0001 C CNN
 	1    4550 5450
@@
 Wire Wire Line
 	7600 1650 7300 1650
-Wire Wire Line
-	7600 1750 7300 1750
 Text Label 7300 1650 2    50   ~ 0
 CAN_H
-Text Label 7300 1750 2    50   ~ 0
-CAN_RES_SW
-Text Label 7300 2050 2    50   ~ 0
-RS485_TERM
 Text Label 7300 1950 2    50   ~ 0
 RS485_B
 Wire Wire Line
+	7600 1950 7300 1950
+Wire Wire Line
+	5850 800  6400 800
+Text Label 6400 800  0    50   ~ 0
+CAN_H
+Wire Wire Line
+	7600 1750 7300 1750
+Text Label 7300 1750 2    50   ~ 0
+CAN_L
+Wire Wire Line
+	5950 1150 6400 1150
+Text Label 6400 1150 0    50   ~ 0
+RS485_B
+Wire Wire Line
 	7600 2050 7300 2050
-Wire Wire Line
-	7600 1950 7300 1950
+Text Label 7300 2050 2    50   ~ 0
+RS485_A
 $EndSCHEMATC

Commit message: --
Parts:
- removed C14, C15: 1u, Capacitor_SMD:C_0805_2012Metric, symbol Device:C
- removed U12, U13: SN74AUP1T34DCK, Package_TO_SOT_SMD:SOT-353_SC-70-5, symbol Logic_LevelTranslator:SN74AUP1T34DCK
Connections:
- net ext_3v3 is gone; now on net GND: J2.3 (Pin_3)
- net ext_RX is gone; now on net U2RX: J2.2 (Pin_2)
- net ext_TX is gone; now on net U2TX: J2.1 (Pin_1)
Changed lines of the file:
@@
-	1    0    0    -1
-$EndComp
-$Comp
-L Logic_LevelTranslator:SN74AUP1T34DCK U12
-U 1 1 5EB1CE3F
-P 3600 4900
-F 0 "U12" H 3900 5250 50  0000 L CNN
-F 1 "SN74AUP1T34DCK" H 3900 5150 50  0000 L CNN
-F 2 "Package_TO_SOT_SMD:SOT-353_SC-70-5" H 3600 4200 50  0001 C CNN
-F 3 "http://www.ti.com/lit/ds/symlink/sn74aup1t34.pdf" H 3600 4300 50  0001 C CNN
-	1    3600 4900
 	1    0    0    -1
 $EndComp
@@
 Wire Wire Line
 	3100 3250 3100 3300
-Wire Wire Line
-	3700 4600 3700 4350
-Text Label 3700 5600 0    50   ~ 0
-ext_3v3
-Text Label 3700 4350 0    50   ~ 0
-ext_3v3
-$Comp
-L power:+3V3 #PWR0153
-U 1 1 5EB26243
-P 3500 4500
-F 0 "#PWR0153" H 3500 4350 50  0001 C CNN
-F 1 "+3V3" H 3515 4673 50  0000 C CNN
-F 2 "" H 3500 4500 50  0001 C CNN
-F 3 "" H 3500 4500 50  0001 C CNN
-	1    3500 4500
-	1    0    0    -1
-$EndComp
-$Comp
-L power:+3V3 #PWR0154
-U 1 1 5EB269EF
-P 3500 5750
-F 0 "#PWR0154" H 3500 5600 50  0001 C CNN
-F 1 "+3V3" H 3515 5923 50  0000 C CNN
-F 2 "" H 3500 5750 50  0001 C CNN
-F 3 "" H 3500 5750 50  0001 C CNN
-	1    3500 5750
-	1    0    0    -1
-$EndComp
-Wire Wire Line
-	3500 4600 3500 4500
-$Comp
-L power:GND #PWR0155
-U 1 1 5EB277E9
-P 3600 6550
-F 0 "#PWR0155" H 3600 6300 50  0001 C CNN
-F 1 "GND" H 3605 6377 50  0000 C CNN
-F 2 "" H 3600 6550 50  0001 C CNN
-F 3 "" H 3600 6550 50  0001 C CNN
-	1    3600 6550
-	1    0    0    -1
-$EndComp
-$Comp
-L power:GND #PWR0156
-U 1 1 5EB28095
-P 3600 5250
-F 0 "#PWR0156" H 3600 5000 50  0001 C CNN
-F 1 "GND" H 3605 5077 50  0000 C CNN
-F 2 "" H 3600 5250 50  0001 C CNN
-F 3 "" H 3600 5250 50  0001 C CNN
-	1    3600 5250
-	1    0    0    -1
-$EndComp
-Wire Wire Line
-	3600 5250 3600 5200
-Text GLabel 4100 4900 2    50   Input ~ 0
-ext_TX
-Text GLabel 4100 6200 2    50   Input ~ 0
-ext_RX
-Wire Wire Line
-	4000 4900 4050 4900
-Text GLabel 3000 4900 0    50   Input ~ 0
+Text GLabel 4250 5350 0    50   Input ~ 0
 U2TX
-Text GLabel 3000 6200 0    50   Input ~ 0
+Text GLabel 4250 5450 0    50   Input ~ 0
 U2RX
-Wire Wire Line
-	3000 4900 3200 4900
 $Comp
 L Device:R R33
@@
 Wire Wire Line
 	2850 3100 3200 3100
-$Comp
-L Device:C C15
-U 1 1 5EB36166
-P 2150 5450
-F 0 "C15" H 2265 5496 50  0000 L CNN
-F 1 "1u" H 2265 5405 50  0000 L CNN
-F 2 "Capacitor_SMD:C_0805_2012Metric" H 2188 5300 50  0001 C CNN
-F 3 "~" H 2150 5450 50  0001 C CNN
-	1    2150 5450
-	1    0    0    -1
-$EndComp
-$Comp
-L Device:C C14
-U 1 1 5EB365C9
-P 1800 5450
-F 0 "C14" H 1915 5496 50  0000 L CNN
-F 1 "1u" H 1915 5405 50  0000 L CNN
-F 2 "Capacitor_SMD:C_0805_2012Metric" H 1838 5300 50  0001 C CNN
-F 3 "~" H 1800 5450 50  0001 C CNN
-	1    1800 5450
-	1    0    0    -1
-$EndComp
-$Comp
-L power:GND #PWR0157
-U 1 1 5EB3682B
-P 1800 5700
-F 0 "#PWR0157" H 1800 5450 50  0001 C CNN
-F 1 "GND" H 1805 5527 50  0000 C CNN
-F 2 "" H 1800 5700 50  0001 C CNN
-F 3 "" H 1800 5700 50  0001 C CNN
-	1    1800 5700
-	1    0    0    -1
-$EndComp
-$Comp
-L power:GND #PWR0158
-U 1 1 5EB36BF0
-P 2150 5700
-F 0 "#PWR0158" H 2150 5450 50  0001 C CNN
-F 1 "GND" H 2155 5527 50  0000 C CNN
-F 2 "" H 2150 5700 50  0001 C CNN
-F 3 "" H 2150 5700 50  0001 C CNN
-	1    2150 5700
-	1    0    0    -1
-$EndComp
-Wire Wire Line
-	2150 5700 2150 5600
-Wire Wire Line
-	1800 5700 1800 5600
-$Comp
-L power:+3V3 #PWR0159
-U 1 1 5EB37F65
-P 1800 5200
-F 0 "#PWR0159" H 1800 5050 50  0001 C CNN
-F 1 "+3V3" H 1815 5373 50  0000 C CNN
-F 2 "" H 1800 5200 50  0001 C CNN
-F 3 "" H 1800 5200 50  0001 C CNN
-	1    1800 5200
-	1    0    0    -1
-$EndComp
-Wire Wire Line
-	1800 5300 1800 5200
-Wire Wire Line
-	2150 5300 2150 5100
-Text Label 2150 5100 0    50   ~ 0
-ext_3v3
-$Comp
-L Logic_LevelTranslator:SN74AUP1T34DCK U13
-U 1 1 5EB1D336
-P 3600 6200
-F 0 "U13" H 3250 5900 50  0000 L CNN
-F 1 "SN74AUP1T34DCK" H 2650 5750 50  0000 L CNN
-F 2 "Package_TO_SOT_SMD:SOT-353_SC-70-5" H 3600 5500 50  0001 C CNN
-F 3 "http://www.ti.com/lit/ds/symlink/sn74aup1t34.pdf" H 3600 5600 50  0001 C CNN
-	1    3600 6200
-	-1   0    0    -1
-$EndComp
-Wire Wire Line
-	3700 5900 3700 5750
-Wire Wire Line
-	3500 5900 3500 5750
-Wire Wire Line
-	4000 6200 4050 6200
-Wire Wire Line
-	3600 6550 3600 6500
-Wire Wire Line
-	3000 6200 3200 6200
 Text Notes 1950 4500 0    118  ~ 0
 RS232 TTL
@@
 $EndComp
 Wire Wire Line
-	4050 5350 4050 4900
-Connection ~ 4050 4900
-Wire Wire Line
-	4050 4900 4100 4900
-Wire Wire Line
-	4050 5450 4050 6200
-Connection ~ 4050 6200
-Wire Wire Line
-	4050 6200 4100 6200
-Wire Wire Line
-	4350 5350 4050 5350
-Wire Wire Line
-	4350 5450 4050 5450
-Wire Wire Line
 	4300 5700 4300 5650
 Wire Wire Line
 	4300 5650 4350 5650
-Wire Wire Line
-	4350 5550 4150 5550
-Wire Wire Line
-	4150 5550 4150 5750
-Wire Wire Line
-	4150 5750 3700 5750
-Connection ~ 3700 5750
-Wire Wire Line
-	3700 5750 3700 5600
 $Comp
 L Connector:Conn_01x02_Male J4
@@
 Text Label 7300 2050 2    50   ~ 0
 RS485_A
+Wire Wire Line
+	4350 5550 4300 5550
+Wire Wire Line
+	4300 5550 4300 5650
+Connection ~ 4300 5650
+Wire Wire Line
+	4250 5450 4350 5450
+Wire Wire Line
+	4250 5350 4350 5350
 $EndSCHEMATC

Commit message: --
Parts:
- renumbered J4 to J3, J5 to J4, R32 to R35, R33 to R36
Changed lines of the file:
@@
 	3100 3300 3200 3300
 $Comp
-L Device:R R32
+L Device:R R35
 U 1 1 5EB1DDEB
 P 5700 800
-F 0 "R32" V 5493 800 50  0000 C CNN
+F 0 "R35" V 5493 800 50  0000 C CNN
 F 1 "120R" V 5584 800 50  0000 C CNN
 F 2 "Resistor_SMD:R_1206_3216Metric" V 5630 800 50  0001 C CNN
@@
 CAN_S
 $Comp
-L power:+3V3 #PWR0149
+L power:+3V3 #PWR052
 U 1 1 5EB23038
 P 3600 1000
-F 0 "#PWR0149" H 3600 850 50  0001 C CNN
+F 0 "#PWR052" H 3600 850 50  0001 C CNN
 F 1 "+3V3" H 3615 1173 50  0000 C CNN
 F 2 "" H 3600 1000 50  0001 C CNN
@@
 	3600 1000 3600 1150
 $Comp
-L power:GND #PWR0150
+L power:GND #PWR053
 U 1 1 5EB23638
 P 3600 2000
-F 0 "#PWR0150" H 3600 1750 50  0001 C CNN
+F 0 "#PWR053" H 3600 1750 50  0001 C CNN
 F 1 "GND" H 3605 1827 50  0000 C CNN
 F 2 "" H 3600 2000 50  0001 C CNN
@@
 	3600 2000 3600 1950
 $Comp
-L power:+3V3 #PWR0151
+L power:+3V3 #PWR054
 U 1 1 5EB23B05
 P 3600 2650
-F 0 "#PWR0151" H 3600 2500 50  0001 C CNN
+F 0 "#PWR054" H 3600 2500 50  0001 C CNN
 F 1 "+3V3" H 3615 2823 50  0000 C CNN
 F 2 "" H 3600 2650 50  0001 C CNN
@@
 $EndComp
 $Comp
-L power:GND #PWR0152
+L power:GND #PWR055
 U 1 1 5EB24292
 P 3600 3850
-F 0 "#PWR0152" H 3600 3600 50  0001 C CNN
+F 0 "#PWR055" H 3600 3600 50  0001 C CNN
 F 1 "GND" H 3605 3677 50  0000 C CNN
 F 2 "" H 3600 3850 50  0001 C CNN
@@
 U2RX
 $Comp
-L Device:R R33
+L Device:R R36
 U 1 1 5EB2BBF3
 P 5800 1150
-F 0 "R33" V 5593 1150 50  0000 C CNN
+F 0 "R36" V 5593 1150 50  0000 C CNN
 F 1 "120R" V 5684 1150 50  0000 C CNN
 F 2 "Resistor_SMD:R_1206_3216Metric" V 5730 1150 50  0001 C CNN
@@
 $EndComp
 $Comp
-L power:GND #PWR0160
+L power:GND #PWR056
 U 1 1 5EB902FC
 P 4300 5700
-F 0 "#PWR0160" H 4300 5450 50  0001 C CNN
+F 0 "#PWR056" H 4300 5450 50  0001 C CNN
 F 1 "GND" H 4305 5527 50  0000 C CNN
 F 2 "" H 4300 5700 50  0001 C CNN
@@
 	4300 5650 4350 5650
 $Comp
-L Connector:Conn_01x02_Male J4
+L Connector:Conn_01x02_Male J3
 U 1 1 5EF64825
 P 7800 1650
-F 0 "J4" H 7908 1831 50  0000 C CNN
+F 0 "J3" H 7908 1831 50  0000 C CNN
 F 1 "Conn_01x02_Male" H 7908 1740 50  0000 C CNN
 F 2 "Connector_PinHeader_2.54mm:PinHeader_1x02_P2.54mm_Vertical" H 7800 1650 50  0001 C CNN
@@
 $EndComp
 $Comp
-L Connector:Conn_01x02_Male J5
+L Connector:Conn_01x02_Male J4
 U 1 1 5EF65E29
 P 7800 1950
-F 0 "J5" H 7954 1762 50  0000 R CNN
+F 0 "J4" H 7954 1762 50  0000 R CNN
 F 1 "Conn_01x02_Male" H 8150 1650 50  0000 R CNN
 F 2 "Connector_PinHeader_2.54mm:PinHeader_1x02_P2.54mm_Vertical" H 7800 1950 50  0001 C CNN
