File: shematic/bldc_drive/io_sheet.sch (KiCad schematic (older format))
At the start: 26 parts, among them J3 Conn_01x04_Male, Q11 2N7002, Q12 2N7002, Q8 BSC440N10NS3G

Commit message: 03.06.2020 21.40 --
Parts:
- added D? (x2): 1N4148W, Diode_SMD:D_SOD-123, symbol Diode:1N4148W
Connections:
- net +12V: now also D?.2 (A); no longer J3.3 (Pin_3), R45.2
- new net: D?.2 (A), J3.3 (Pin_3)
- new net: D?.1 (K), D?.1 (K), R45.2
Changed lines of the file:
@@
 $EndComp
-Wire Wire Line
-	9100 1250 9750 1250
-Wire Wire Line
-	9100 1250 9100 800
-Connection ~ 9100 1250
-Wire Wire Line
-	9100 1600 9100 1250
 Wire Wire Line
 	9450 2700 9450 2600
@@
 Wire Wire Line
 	1550 4800 1550 4500
+$Comp
+L Diode:1N4148W D?
+U 1 1 5EDCFF6A
+P 9100 1000
+F 0 "D?" V 9100 1400 50  0000 R CNN
+F 1 "1N4148W" V 9000 1450 50  0000 R CNN
+F 2 "Diode_SMD:D_SOD-123" H 9100 825 50  0001 C CNN
+F 3 "https://www.vishay.com/docs/85748/1n4148w.pdf" H 9100 1000 50  0001 C CNN
+	1    9100 1000
+	0    -1   -1   0
+$EndComp
+Wire Wire Line
+	9100 850  9100 800
+Wire Wire Line
+	9100 1150 9100 1250
+$Comp
+L Diode:1N4148W D?
+U 1 1 5EDD81B6
+P 9250 1250
+F 0 "D?" V 9250 1650 50  0000 R CNN
+F 1 "1N4148W" V 9150 1700 50  0000 R CNN
+F 2 "Diode_SMD:D_SOD-123" H 9250 1075 50  0001 C CNN
+F 3 "https://www.vishay.com/docs/85748/1n4148w.pdf" H 9250 1250 50  0001 C CNN
+	1    9250 1250
+	1    0    0    -1
+$EndComp
+Connection ~ 9100 1250
+Wire Wire Line
+	9100 1250 9100 1600
+Wire Wire Line
+	9400 1250 9750 1250
 $EndSCHEMATC

Commit message: 11.06.2020 21.40 --
Parts:
- removed Q8: BSC440N10NS3G, Package_TO_SOT_SMD:TDSON-8-1, symbol Transistor_FET:BSC440N10NS3G
- added Q8: FDS6930B, Package_SO:SOIC-8_3.9x4.9mm_P1.27mm, symbol Transistor_FET:FDS6930B
- C16, C17, C18: footprint (none) -> Capacitor_SMD:C_0603_1608Metric
- C20, C21: footprint (none) -> Capacitor_SMD:C_0805_2012Metric
- J3: footprint (none) -> Connector_PinHeader_2.54mm:PinHeader_1x04_P2.54mm_Vertical
- R34, R36, R37, R39, R40, R41, R42, R45, R46, R47, R48: footprint (none) -> Resistor_SMD:R_0603_1608Metric
- gave numbers to parts that had none: 2
Connections:
- net GND: now also Q8.1 (S1)
- net OD_OUT_1: now also Q8.7 (D1), Q8.8 (D1)
- net at R34.1: now also Q8.2 (G1)
Changed lines of the file:
@@
 F 0 "C16" H 2615 2596 50  0000 L CNN
 F 1 "100n" H 2615 2505 50  0000 L CNN
-F 2 "" H 2538 2400 50  0001 C CNN
+F 2 "Capacitor_SMD:C_0603_1608Metric" H 2538 2400 50  0001 C CNN
 F 3 "~" H 2500 2550 50  0001 C CNN
 	1    2500 2550
@@
 F 0 "R36" H 2730 2054 50  0000 R CNN
 F 1 "4k7" H 2730 2145 50  0000 R CNN
-F 2 "" V 2730 2100 50  0001 C CNN
+F 2 "Resistor_SMD:R_0603_1608Metric" V 2730 2100 50  0001 C CNN
 F 3 "~" H 2800 2100 50  0001 C CNN
 	1    2800 2100
@@
 F 0 "R37" H 2730 2504 50  0000 R CNN
 F 1 "2k2" H 2730 2595 50  0000 R CNN
-F 2 "" V 2730 2550 50  0001 C CNN
+F 2 "Resistor_SMD:R_0603_1608Metric" V 2730 2550 50  0001 C CNN
 F 3 "~" H 2800 2550 50  0001 C CNN
 	1    2800 2550
@@
 F 0 "J3" H 10058 1431 50  0000 C CNN
 F 1 "Conn_01x04_Male" H 10058 1340 50  0000 C CNN
-F 2 "" H 9950 1150 50  0001 C CNN
+F 2 "Connector_PinHeader_2.54mm:PinHeader_1x04_P2.54mm_Vertical" H 9950 1150 50  0001 C CNN
 F 3 "~" H 9950 1150 50  0001 C CNN
 	1    9950 1150
@@
 F 0 "C20" H 8315 2346 50  0000 L CNN
 F 1 "1u" H 8315 2255 50  0000 L CNN
-F 2 "" H 8238 2150 50  0001 C CNN
+F 2 "Capacitor_SMD:C_0805_2012Metric" H 8238 2150 50  0001 C CNN
 F 3 "~" H 8200 2300 50  0001 C CNN
 	1    8200 2300
@@
 F 0 "C21" H 8665 2346 50  0000 L CNN
 F 1 "1u" H 8665 2255 50  0000 L CNN
-F 2 "" H 8588 2150 50  0001 C CNN
+F 2 "Capacitor_SMD:C_0805_2012Metric" H 8588 2150 50  0001 C CNN
 F 3 "~" H 8550 2300 50  0001 C CNN
 	1    8550 2300
@@
 F 0 "R46" H 9030 2154 50  0000 R CNN
 F 1 "2k2" H 9030 2245 50  0000 R CNN
-F 2 "" V 9030 2200 50  0001 C CNN
+F 2 "Resistor_SMD:R_0603_1608Metric" V 9030 2200 50  0001 C CNN
 F 3 "~" H 9100 2200 50  0001 C CNN
 	1    9100 2200
@@
 F 0 "R45" H 9030 1704 50  0000 R CNN
 F 1 "4k7" H 9030 1795 50  0000 R CNN
-F 2 "" V 9030 1750 50  0001 C CNN
+F 2 "Resistor_SMD:R_0603_1608Metric" V 9030 1750 50  0001 C CNN
 F 3 "~" H 9100 1750 50  0001 C CNN
 	1    9100 1750
@@
 F 0 "R48" H 9380 2154 50  0000 R CNN
 F 1 "2k2" H 9380 2245 50  0000 R CNN
-F 2 "" V 9380 2200 50  0001 C CNN
+F 2 "Resistor_SMD:R_0603_1608Metric" V 9380 2200 50  0001 C CNN
 F 3 "~" H 9450 2200 50  0001 C CNN
 	1    9450 2200
@@
 F 0 "R47" H 9380 1704 50  0000 R CNN
 F 1 "4k7" H 9380 1795 50  0000 R CNN
-F 2 "" V 9380 1750 50  0001 C CNN
+F 2 "Resistor_SMD:R_0603_1608Metric" V 9380 1750 50  0001 C CNN
 F 3 "~" H 9450 1750 50  0001 C CNN
 	1    9450 1750
 	-1   0    0    1
-$EndComp
-$Comp
-L Transistor_FET:BSC440N10NS3G Q8
-U 1 1 5ED23A91
-P 1450 5000
-F 0 "Q8" H 1655 5000 50  0000 L CNN
-F 1 "BSC440N10NS3G" H 1654 4955 50  0001 L CNN
-F 2 "Package_TO_SOT_SMD:TDSON-8-1" H 1650 4925 50  0001 L CIN
-F 3 "http://www.infineon.com/dgdl/Infineon-BSC440N10NS3-DS-v02_04-en.pdf?fileId=db3a30432239cccd0122604520d47f56" V 1450 5000 50  0001 L CNN
-	1    1450 5000
-	1    0    0    -1
 $EndComp
 $Comp
@@
 F 0 "R34" V 893 5000 50  0000 C CNN
 F 1 "R" V 984 5000 50  0000 C CNN
-F 2 "" V 1030 5000 50  0001 C CNN
+F 2 "Resistor_SMD:R_0603_1608Metric" V 1030 5000 50  0001 C CNN
 F 3 "~" H 1100 5000 50  0001 C CNN
 	1    1100 5000
@@
 F 0 "R40" H 3130 4404 50  0000 R CNN
 F 1 "10k" H 3130 4495 50  0000 R CNN
-F 2 "" V 3130 4450 50  0001 C CNN
+F 2 "Resistor_SMD:R_0603_1608Metric" V 3130 4450 50  0001 C CNN
 F 3 "~" H 3200 4450 50  0001 C CNN
 	1    3200 4450
@@
 F 0 "R42" H 4530 4404 50  0000 R CNN
 F 1 "10k" H 4530 4495 50  0000 R CNN
-F 2 "" V 4530 4450 50  0001 C CNN
+F 2 "Resistor_SMD:R_0603_1608Metric" V 4530 4450 50  0001 C CNN
 F 3 "~" H 4600 4450 50  0001 C CNN
 	1    4600 4450
@@
 F 0 "C18" H 4015 5146 50  0000 L CNN
 F 1 "100n" H 4015 5055 50  0000 L CNN
-F 2 "" H 3938 4950 50  0001 C CNN
+F 2 "Capacitor_SMD:C_0603_1608Metric" H 3938 4950 50  0001 C CNN
 F 3 "~" H 3900 5100 50  0001 C CNN
 	1    3900 5100
@@
 F 0 "C17" H 2615 5146 50  0000 L CNN
 F 1 "100n" H 2615 5055 50  0000 L CNN
-F 2 "" H 2538 4950 50  0001 C CNN
+F 2 "Capacitor_SMD:C_0603_1608Metric" H 2538 4950 50  0001 C CNN
 F 3 "~" H 2500 5100 50  0001 C CNN
 	1    2500 5100
@@
 F 0 "R41" H 3830 4404 50  0000 R CNN
 F 1 "10k" H 3830 4495 50  0000 R CNN
-F 2 "" V 3830 4450 50  0001 C CNN
+F 2 "Resistor_SMD:R_0603_1608Metric" V 3830 4450 50  0001 C CNN
 F 3 "~" H 3900 4450 50  0001 C CNN
 	1    3900 4450
@@
 F 0 "R39" H 2430 4404 50  0000 R CNN
 F 1 "10k" H 2430 4495 50  0000 R CNN
-F 2 "" V 2430 4450 50  0001 C CNN
+F 2 "Resistor_SMD:R_0603_1608Metric" V 2430 4450 50  0001 C CNN
 F 3 "~" H 2500 4450 50  0001 C CNN
 	1    2500 4450
@@
 	1550 4800 1550 4500
 $Comp
-L Diode:1N4148W D?
+L Diode:1N4148W D9
 U 1 1 5EDCFF6A
 P 9100 1000
-F 0 "D?" V 9100 1400 50  0000 R CNN
+F 0 "D9" V 9100 1400 50  0000 R CNN
 F 1 "1N4148W" V 9000 1450 50  0000 R CNN
 F 2 "Diode_SMD:D_SOD-123" H 9100 825 50  0001 C CNN
@@
 	9100 1150 9100 1250
 $Comp
-L Diode:1N4148W D?
+L Diode:1N4148W D10
 U 1 1 5EDD81B6
 P 9250 1250
-F 0 "D?" V 9250 1650 50  0000 R CNN
+F 0 "D10" V 9250 1650 50  0000 R CNN
 F 1 "1N4148W" V 9150 1700 50  0000 R CNN
 F 2 "Diode_SMD:D_SOD-123" H 9250 1075 50  0001 C CNN
@@
 Wire Wire Line
 	9400 1250 9750 1250
+$Comp
+L Transistor_FET:FDS6930B Q8
+U 1 1 5EFDAAAA
+P 1450 5000
+F 0 "Q8" H 1655 5046 50  0000 L CNN
+F 1 "FDS6930B" H 1655 4955 50  0000 L CNN
+F 2 "Package_SO:SOIC-8_3.9x4.9mm_P1.27mm" H 1650 4925 50  0001 L CIN
+F 3 "http://www.onsemi.com/pub/Collateral/FDS6930B-D.PDF" H 1450 5000 50  0001 L CNN
+	1    1450 5000
+	1    0    0    -1
+$EndComp
 $EndSCHEMATC

Commit message: --
Parts:
- removed C16, C17, C18: 100n, Capacitor_SMD:C_0603_1608Metric, symbol Device:C
- removed D12, D13, D8: DZ2S033X0L, Diode_SMD:D_SOD-523, symbol Diode:DZ2S033X0L
- removed D6: 1N4148W, Diode_SMD:D_SOD-123, symbol Diode:1N4148W
- removed Q11, Q12: 2N7002, Package_TO_SOT_SMD:SOT-23, symbol Transistor_FET:2N7002
- removed Q8: FDS6930B, Package_SO:SOIC-8_3.9x4.9mm_P1.27mm, symbol Transistor_FET:FDS6930B
- removed R34: R, Resistor_SMD:R_0603_1608Metric, symbol Device:R
- removed R36: 4k7, Resistor_SMD:R_0603_1608Metric, symbol Device:R
- removed R37: 2k2, Resistor_SMD:R_0603_1608Metric, symbol Device:R
- removed R39, R40, R41, R42: 10k, Resistor_SMD:R_0603_1608Metric, symbol Device:R

Commit message: --
Parts:
- renumbered C20 to C12, C21 to C13, D14 to D7, D16 to D8, J3 to J5, R45 to R37, R46 to R38, R47 to R39, R48 to R40
Changed lines of the file:
@@
 P 9950 1150
 AR Path="/5EB1ABF5/5ED191D1" Ref="J?"  Part="1"
-AR Path="/5ED063DC/5ED191D1" Ref="J3"  Part="1"
-F 0 "J3" H 10058 1431 50  0000 C CNN
+AR Path="/5ED063DC/5ED191D1" Ref="J5"  Part="1"
+F 0 "J5" H 10058 1431 50  0000 C CNN
 F 1 "Conn_01x04_Male" H 10058 1340 50  0000 C CNN
 F 2 "Connector_PinHeader_2.54mm:PinHeader_1x04_P2.54mm_Vertical" H 9950 1150 50  0001 C CNN
@@
 P 8200 2300
 AR Path="/5EB1ABF5/5ED191E8" Ref="C?"  Part="1"
-AR Path="/5ED063DC/5ED191E8" Ref="C20"  Part="1"
-F 0 "C20" H 8315 2346 50  0000 L CNN
+AR Path="/5ED063DC/5ED191E8" Ref="C12"  Part="1"
+F 0 "C12" H 8315 2346 50  0000 L CNN
 F 1 "1u" H 8315 2255 50  0000 L CNN
 F 2 "Capacitor_SMD:C_0805_2012Metric" H 8238 2150 50  0001 C CNN
@@
 P 8550 2300
 AR Path="/5EB1ABF5/5ED191EE" Ref="C?"  Part="1"
-AR Path="/5ED063DC/5ED191EE" Ref="C21"  Part="1"
-F 0 "C21" H 8665 2346 50  0000 L CNN
+AR Path="/5ED063DC/5ED191EE" Ref="C13"  Part="1"
+F 0 "C13" H 8665 2346 50  0000 L CNN
 F 1 "1u" H 8665 2255 50  0000 L CNN
 F 2 "Capacitor_SMD:C_0805_2012Metric" H 8588 2150 50  0001 C CNN
@@
 P 8850 2300
 AR Path="/5EB1ABF5/5ED191FF" Ref="D?"  Part="1"
-AR Path="/5ED063DC/5ED191FF" Ref="D16"  Part="1"
-F 0 "D16" V 8750 2200 50  0000 L CNN
+AR Path="/5ED063DC/5ED191FF" Ref="D8"  Part="1"
+F 0 "D8" V 8750 2200 50  0000 L CNN
 F 1 "DZ2S033X0L" V 9350 2350 50  0001 L CNN
 F 2 "Diode_SMD:D_SOD-523" H 8850 2125 50  0001 C CNN
@@
 P 8000 2300
 AR Path="/5EB1ABF5/5ED19205" Ref="D?"  Part="1"
-AR Path="/5ED063DC/5ED19205" Ref="D14"  Part="1"
-F 0 "D14" V 7900 2150 50  0000 L CNN
+AR Path="/5ED063DC/5ED19205" Ref="D7"  Part="1"
+F 0 "D7" V 7900 2150 50  0000 L CNN
 F 1 "DZ2S033X0L" V 8500 2150 50  0001 L CNN
 F 2 "Diode_SMD:D_SOD-523" H 8000 2125 50  0001 C CNN
@@
 P 9450 2700
 AR Path="/5EB1ABF5/5ED19212" Ref="#PWR?"  Part="1"
-AR Path="/5ED063DC/5ED19212" Ref="#PWR0162"  Part="1"
-F 0 "#PWR0162" H 9450 2450 50  0001 C CNN
+AR Path="/5ED063DC/5ED19212" Ref="#PWR058"  Part="1"
+F 0 "#PWR058" H 9450 2450 50  0001 C CNN
 F 1 "GND" H 9455 2527 50  0000 C CNN
 F 2 "" H 9450 2700 50  0001 C CNN
@@
 P 9100 800
 AR Path="/5EB1ABF5/5ED1921C" Ref="#PWR?"  Part="1"
-AR Path="/5ED063DC/5ED1921C" Ref="#PWR0163"  Part="1"
-F 0 "#PWR0163" H 9100 650 50  0001 C CNN
+AR Path="/5ED063DC/5ED1921C" Ref="#PWR057"  Part="1"
+F 0 "#PWR057" H 9100 650 50  0001 C CNN
 F 1 "+12V" H 9115 973 50  0000 C CNN
 F 2 "" H 9100 800 50  0001 C CNN
@@
 P 9100 2200
 AR Path="/5EB1ABF5/5ED19228" Ref="R?"  Part="1"
-AR Path="/5ED063DC/5ED19228" Ref="R46"  Part="1"
-F 0 "R46" H 9030 2154 50  0000 R CNN
+AR Path="/5ED063DC/5ED19228" Ref="R38"  Part="1"
+F 0 "R38" H 9030 2154 50  0000 R CNN
 F 1 "2k2" H 9030 2245 50  0000 R CNN
 F 2 "Resistor_SMD:R_0603_1608Metric" V 9030 2200 50  0001 C CNN
@@
 P 9100 1750
 AR Path="/5EB1ABF5/5ED1922F" Ref="R?"  Part="1"
-AR Path="/5ED063DC/5ED1922F" Ref="R45"  Part="1"
-F 0 "R45" H 9030 1704 50  0000 R CNN
+AR Path="/5ED063DC/5ED1922F" Ref="R37"  Part="1"
+F 0 "R37" H 9030 1704 50  0000 R CNN
 F 1 "4k7" H 9030 1795 50  0000 R CNN
 F 2 "Resistor_SMD:R_0603_1608Metric" V 9030 1750 50  0001 C CNN
@@
 P 9450 2200
 AR Path="/5EB1ABF5/5ED19235" Ref="R?"  Part="1"
-AR Path="/5ED063DC/5ED19235" Ref="R48"  Part="1"
-F 0 "R48" H 9380 2154 50  0000 R CNN
+AR Path="/5ED063DC/5ED19235" Ref="R40"  Part="1"
+F 0 "R40" H 9380 2154 50  0000 R CNN
 F 1 "2k2" H 9380 2245 50  0000 R CNN
 F 2 "Resistor_SMD:R_0603_1608Metric" V 9380 2200 50  0001 C CNN
@@
 P 9450 1750
 AR Path="/5EB1ABF5/5ED1923B" Ref="R?"  Part="1"
-AR Path="/5ED063DC/5ED1923B" Ref="R47"  Part="1"
-F 0 "R47" H 9380 1704 50  0000 R CNN
+AR Path="/5ED063DC/5ED1923B" Ref="R39"  Part="1"
+F 0 "R39" H 9380 1704 50  0000 R CNN
 F 1 "4k7" H 9380 1795 50  0000 R CNN
 F 2 "Resistor_SMD:R_0603_1608Metric" V 9380 1750 50  0001 C CNN
