File: shematic/bldc_drive/power_conv.sch (KiCad schematic (older format))
At the start: 18 parts

Commit message: 11.06.2020 21.40 --
Parts:
- added C19: 2u2, Capacitor_SMD:C_1206_3216Metric, symbol Device:C
- added C30, C31: C, Capacitor_SMD:C_0805_2012Metric, symbol Device:C
- added C32: CP, Capacitor_SMD:C_Elec_8x5.4, symbol Device:CP
- added C33: 2200uf, Capacitor_THT:CP_Radial_D35.0mm_P10.00mm_SnapIn, symbol Device:CP
- added D15: D_Zener, Diode_SMD:D_SMB, symbol Device:D_Zener
- added H2, H3, H4, H5, H6, H7, H8: MountingHole_Pad, MountingHole:MountingHole_3.5mm_Pad_Via, symbol Mechanical:MountingHole_Pad
- added L1, L2: INDUCTOR, Inductor_THT:L_Axial_L30.0mm_D8.0mm_P35.56mm_Horizontal_Fastron_77A, symbol pspice:INDUCTOR
- added U14: uA7812, Package_TO_SOT_THT:TO-220-3_Horizontal_TabDown, symbol Regulator_Linear:uA7812
- added U15: AP1117-33, Package_TO_SOT_SMD:SOT-223-3_TabPin2, symbol Regulator_Linear:AP1117-33
- C22: renamed from C?; value C -> 1u; footprint (none) -> Capacitor_SMD:C_1206_3216Metric
- C23: renamed from C?; value CP -> 2200uf; footprint (none) -> Capacitor_THT:CP_Radial_D35.0mm_P10.00mm_SnapIn
- C24, C25: renamed from C?; footprint (none) -> Capacitor_SMD:C_0603_1608Metric
- C26, C27, C28: renamed from C?; footprint (none) -> Capacitor_SMD:C_0805_2012Metric
- C29: renamed from C?; footprint (none) -> Capacitor_SMD:C_Elec_8x6.2
- H1: renamed from H?; footprint (none) -> MountingHole:MountingHole_3.5mm_Pad_Via
- IC1: renamed from IC?; footprint SOP50P490X110-11N -> msop10:SOP50P490X110-11N
- L3: renamed from L?; footprint (none) -> Inductor_SMD:L_Bourns-SRN6028
- R38, R43, R44, R50, R51: renamed from R?; footprint (none) -> Resistor_SMD:R_0603_1608Metric
- R49: renamed from R?; footprint (none) -> Resistor_SMD:R_0805_2012Metric
- gave numbers to parts that had none: 1
Connections:
- net labels added: +12V, +3V3, +V_POW
- wire segments 65 -> 113
Other:
- moved on the sheet: C22, H1

Commit message: --
Parts:
- removed C25: 100n, Capacitor_SMD:C_0603_1608Metric, symbol Device:C
- removed C26, C27, C28: C, Capacitor_SMD:C_0805_2012Metric, symbol Device:C
- removed C29: CP, Capacitor_SMD:C_Elec_8x6.2, symbol Device:CP
- removed D11: B340, Diode_SMD:D_SMC, symbol Diode:B340
- removed H3, H4, H6: MountingHole_Pad, MountingHole:MountingHole_3.5mm_Pad_Via, symbol Mechanical:MountingHole_Pad
- removed IC1: TPS54140ADGQR, msop10:SOP50P490X110-11N, symbol tps54140:TPS54140ADGQR
- removed L3: INDUCTOR, Inductor_SMD:L_Bourns-SRN6028, symbol pspice:INDUCTOR
- removed R38, R43, R44, R50, R51: R, Resistor_SMD:R_0603_1608Metric, symbol Device:R
- removed R49: R, Resistor_SMD:R_0805_2012Metric, symbol Device:R
- C23, C33: footprint Capacitor_THT:CP_Radial_D35.0mm_P10.00mm_SnapIn -> Capacitor_THT:CP_Radial_D18.0mm_P7.50mm
- C24: value C -> 1u; footprint Capacitor_SMD:C_0603_1608Metric -> Capacitor_SMD:C_1206_3216Metric
- L1, L2: footprint Inductor_THT:L_Axial_L30.0mm_D8.0mm_P35.56mm_Horizontal_Fastron_77A -> Inductor_THT:L_Axial_L20.0mm_D8.0mm_P25.40mm_Horizontal
- U14: footprint Package_TO_SOT_THT:TO-220-3_Horizontal_TabDown -> Package_TO_SOT_THT:TO-220-3_Vertical
Connections:
- wire segments 113 -> 42
Other:
- moved on the sheet: C30, C31, C32, D15, H1, H7, H8, U14, U15

Commit message: 29.08.20
Parts:
- removed H7, H8: MountingHole_Pad, MountingHole:MountingHole_3.5mm_Pad_Via, symbol Mechanical:MountingHole_Pad
Changed lines of the file:
@@
 	1    0    0    -1
 $EndComp
-Wire Wire Line
-	4550 2500 4650 2500
-$Comp
-L Mechanical:MountingHole_Pad H7
-U 1 1 5EF90967
-P 3950 2050
-F 0 "H7" H 4050 2200 50  0000 L CNN
-F 1 "MountingHole_Pad" H 4050 2008 50  0001 L CNN
-F 2 "MountingHole:MountingHole_3.5mm_Pad_Via" H 3950 2050 50  0001 C CNN
-F 3 "~" H 3950 2050 50  0001 C CNN
-	1    3950 2050
-	1    0    0    -1
-$EndComp
-$Comp
-L Mechanical:MountingHole_Pad H8
-U 1 1 5EF915A9
-P 4650 2050
-F 0 "H8" H 4750 2200 50  0000 L CNN
-F 1 "MountingHole_Pad" H 4750 2008 50  0001 L CNN
-F 2 "MountingHole:MountingHole_3.5mm_Pad_Via" H 4650 2050 50  0001 C CNN
-F 3 "~" H 4650 2050 50  0001 C CNN
-	1    4650 2050
-	1    0    0    -1
-$EndComp
-Wire Wire Line
-	3950 2150 3950 2500
-Connection ~ 3950 2500
-Wire Wire Line
-	4650 2150 4650 2500
-Connection ~ 4650 2500
 $Comp
 L Device:D_Zener D15
@@
 $EndComp
 Wire Wire Line
-	4650 2500 5200 2500
-Wire Wire Line
 	1300 950  1300 1200
 Wire Wire Line
@@
 	1    0    0    -1
 $EndComp
+Wire Wire Line
+	4550 2500 5200 2500
 $EndSCHEMATC

Commit message: --
Parts:
- removed C32: CP, Capacitor_SMD:C_Elec_8x5.4, symbol Device:CP
- H2: footprint MountingHole:MountingHole_3.5mm_Pad_Via -> MountingHole:MountingHole_4.3mm_M4_Pad_Via
- L1, L2: footprint Inductor_THT:L_Axial_L20.0mm_D8.0mm_P25.40mm_Horizontal -> Inductor_THT:L_Axial_L16.0mm_D6.3mm_P20.32mm_Horizontal_Fastron_VHBCC
Changed lines of the file:
@@
 F 0 "L2" H 2300 1865 50  0000 C CNN
 F 1 "INDUCTOR" H 2300 1774 50  0000 C CNN
-F 2 "Inductor_THT:L_Axial_L20.0mm_D8.0mm_P25.40mm_Horizontal" H 2300 1650 50  0001 C CNN
+F 2 "Inductor_THT:L_Axial_L16.0mm_D6.3mm_P20.32mm_Horizontal_Fastron_VHBCC" H 2300 1650 50  0001 C CNN
 F 3 "~" H 2300 1650 50  0001 C CNN
 	1    2300 1650
@@
 F 0 "L1" H 1300 1815 50  0000 C CNN
 F 1 "INDUCTOR" H 1300 1724 50  0000 C CNN
-F 2 "Inductor_THT:L_Axial_L20.0mm_D8.0mm_P25.40mm_Horizontal" H 1300 1600 50  0001 C CNN
+F 2 "Inductor_THT:L_Axial_L16.0mm_D6.3mm_P20.32mm_Horizontal_Fastron_VHBCC" H 1300 1600 50  0001 C CNN
 F 3 "~" H 1300 1600 50  0001 C CNN
 	1    1300 1600
@@
 	1    0    0    -1
 $EndComp
-$Comp
-L Device:CP C32
-U 1 1 5EE775F3
-P 6600 2750
-F 0 "C32" H 6718 2796 50  0000 L CNN
-F 1 "CP" H 6718 2705 50  0000 L CNN
-F 2 "Capacitor_SMD:C_Elec_8x5.4" H 6638 2600 50  0001 C CNN
-F 3 "~" H 6600 2750 50  0001 C CNN
-	1    6600 2750
-	1    0    0    -1
-$EndComp
 Wire Wire Line
 	5200 2600 5200 2500
@@
 	6050 2500 6250 2500
 Wire Wire Line
-	6600 2500 6600 2600
-Wire Wire Line
 	6250 2600 6250 2500
 Connection ~ 6250 2500
@@
 Wire Wire Line
 	5200 2900 5750 2900
-Wire Wire Line
-	6600 2900 6250 2900
 Wire Wire Line
 	6250 2900 5750 2900
@@
 	6900 2850 6900 2900
 Wire Wire Line
-	6900 2900 6600 2900
-Connection ~ 6600 2900
-Wire Wire Line
 	6600 2500 6900 2500
 Wire Wire Line
@@
 F 0 "H2" H 3100 3600 50  0000 L CNN
 F 1 "MountingHole_Pad" H 3100 3408 50  0001 L CNN
-F 2 "MountingHole:MountingHole_3.5mm_Pad_Via" H 3000 3450 50  0001 C CNN
+F 2 "MountingHole:MountingHole_4.3mm_M4_Pad_Via" H 3000 3450 50  0001 C CNN
 F 3 "~" H 3000 3450 50  0001 C CNN
 	1    3000 3450
@@
 Wire Wire Line
 	4550 2500 5200 2500
+Wire Wire Line
+	6250 2900 6900 2900
 $EndSCHEMATC

Commit message: --
Parts:
- renumbered C22 to C14, C19 to C15, C33 to C16, C23 to C17, C24 to C18, C30 to C19, C31 to C20, D15 to D11, H1 to H4, H2 to H6, U14 to U12, U15 to U13
Changed lines of the file:
@@
 $EndDescr
 $Comp
-L Mechanical:MountingHole_Pad H1
+L Mechanical:MountingHole_Pad H4
 U 1 1 5EDC6E08
 P 1300 850
-F 0 "H1" H 1400 1000 50  0000 L CNN
+F 0 "H4" H 1400 1000 50  0000 L CNN
 F 1 "MountingHole_Pad" H 1400 808 50  0001 L CNN
 F 2 "MountingHole:MountingHole_3.5mm_Pad_Via" H 1300 850 50  0001 C CNN
@@
 $EndComp
 $Comp
-L Device:CP C23
+L Device:CP C17
 U 1 1 5EDCC0C3
 P 2150 3000
-F 0 "C23" H 2268 3046 50  0000 L CNN
+F 0 "C17" H 2268 3046 50  0000 L CNN
 F 1 "2200uf" H 2268 2955 50  0000 L CNN
 F 2 "Capacitor_THT:CP_Radial_D18.0mm_P7.50mm" H 2188 2850 50  0001 C CNN
@@
 $EndComp
 $Comp
-L Device:C C22
+L Device:C C14
 U 1 1 5EDCC9D3
 P 1500 3000
-F 0 "C22" H 1615 3046 50  0000 L CNN
+F 0 "C14" H 1615 3046 50  0000 L CNN
 F 1 "1u" H 1615 2955 50  0000 L CNN
 F 2 "Capacitor_SMD:C_1206_3216Metric" H 1538 2850 50  0001 C CNN
@@
 	1300 1350 1300 1200
 $Comp
-L power:GND #PWR04
+L power:GND #PWR059
 U 1 1 5EE6767B
 P 1300 3500
-F 0 "#PWR04" H 1300 3250 50  0001 C CNN
+F 0 "#PWR059" H 1300 3250 50  0001 C CNN
 F 1 "GND" H 1305 3327 50  0000 C CNN
 F 2 "" H 1300 3500 50  0001 C CNN
@@
 	1300 3500 1300 1850
 $Comp
-L Device:C C19
+L Device:C C15
 U 1 1 5EE6CFDC
 P 1800 1200
-F 0 "C19" H 1915 1246 50  0000 L CNN
+F 0 "C15" H 1915 1246 50  0000 L CNN
 F 1 "2u2" H 1915 1155 50  0000 L CNN
 F 2 "Capacitor_SMD:C_1206_3216Metric" H 1838 1050 50  0001 C CNN
@@
 Connection ~ 2300 1200
 $Comp
-L Regulator_Linear:AP1117-33 U15
+L Regulator_Linear:AP1117-33 U13
 U 1 1 5EE72DF7
 P 5750 2500
-F 0 "U15" H 5750 2742 50  0000 C CNN
+F 0 "U13" H 5750 2742 50  0000 C CNN
 F 1 "AP1117-33" H 5750 2651 50  0000 C CNN
 F 2 "Package_TO_SOT_SMD:SOT-223-3_TabPin2" H 5750 2700 50  0001 C CNN
@@
 $EndComp
 $Comp
-L power:+12V #PWR09
+L power:+12V #PWR063
 U 1 1 5EE7383E
 P 5200 2400
-F 0 "#PWR09" H 5200 2250 50  0001 C CNN
+F 0 "#PWR063" H 5200 2250 50  0001 C CNN
 F 1 "+12V" H 5215 2573 50  0000 C CNN
 F 2 "" H 5200 2400 50  0001 C CNN
@@
 	5200 2500 5450 2500
 $Comp
-L power:GND #PWR010
+L power:GND #PWR064
 U 1 1 5EE76A4E
 P 5750 2900
-F 0 "#PWR010" H 5750 2650 50  0001 C CNN
+F 0 "#PWR064" H 5750 2650 50  0001 C CNN
 F 1 "GND" H 5755 2727 50  0000 C CNN
 F 2 "" H 5750 2900 50  0001 C CNN
@@
 $EndComp
 $Comp
-L Device:C C30
+L Device:C C19
 U 1 1 5EE76E06
 P 5200 2750
-F 0 "C30" H 5315 2796 50  0000 L CNN
+F 0 "C19" H 5315 2796 50  0000 L CNN
 F 1 "C" H 5315 2705 50  0000 L CNN
 F 2 "Capacitor_SMD:C_0805_2012Metric" H 5238 2600 50  0001 C CNN
@@
 $EndComp
 $Comp
-L Device:C C31
+L Device:C C20
 U 1 1 5EE77226
 P 6250 2750
-F 0 "C31" H 6365 2796 50  0000 L CNN
+F 0 "C20" H 6365 2796 50  0000 L CNN
 F 1 "C" H 6365 2705 50  0000 L CNN
 F 2 "Capacitor_SMD:C_0805_2012Metric" H 6288 2600 50  0001 C CNN
@@
 	5750 2800 5750 2900
 $Comp
-L power:+3V3 #PWR011
+L power:+3V3 #PWR065
 U 1 1 5EE8EF0A
 P 6600 2400
-F 0 "#PWR011" H 6600 2250 50  0001 C CNN
+F 0 "#PWR065" H 6600 2250 50  0001 C CNN
 F 1 "+3V3" H 6615 2573 50  0000 C CNN
 F 2 "" H 6600 2400 50  0001 C CNN
@@
 Connection ~ 6600 2500
 $Comp
-L Regulator_Linear:uA7812 U14
+L Regulator_Linear:uA7812 U12
 U 1 1 5EF89054
 P 4250 2500
-F 0 "U14" H 4250 2742 50  0000 C CNN
+F 0 "U12" H 4250 2742 50  0000 C CNN
 F 1 "uA7812" H 4250 2651 50  0000 C CNN
 F 2 "Package_TO_SOT_THT:TO-220-3_Vertical" H 4275 2350 50  0001 L CIN
@@
 $EndComp
 $Comp
-L power:GND #PWR06
+L power:GND #PWR062
 U 1 1 5EF8C17E
 P 4250 2800
-F 0 "#PWR06" H 4250 2550 50  0001 C CNN
+F 0 "#PWR062" H 4250 2550 50  0001 C CNN
 F 1 "GND" H 4255 2627 50  0000 C CNN
 F 2 "" H 4250 2800 50  0001 C CNN
@@
 $EndComp
 $Comp
-L Device:D_Zener D15
+L Device:D_Zener D11
 U 1 1 5EF9F773
 P 6900 2700
-F 0 "D15" V 6854 2779 50  0000 L CNN
+F 0 "D11" V 6854 2779 50  0000 L CNN
 F 1 "D_Zener" V 6945 2779 50  0000 L CNN
 F 2 "Diode_SMD:D_SMB" H 6900 2700 50  0001 C CNN
@@
 	6900 2500 6900 2550
 $Comp
-L Device:CP C33
+L Device:CP C16
 U 1 1 5EFBC0B5
 P 1800 3000
-F 0 "C33" H 1918 3046 50  0000 L CNN
+F 0 "C16" H 1918 3046 50  0000 L CNN
 F 1 "2200uf" H 1918 2955 50  0000 L CNN
 F 2 "Capacitor_THT:CP_Radial_D18.0mm_P7.50mm" H 1838 2850 50  0001 C CNN
@@
 Connection ~ 3100 2500
 $Comp
-L power:GND #PWR0164
+L power:GND #PWR060
 U 1 1 5F377594
 P 1800 3450
-F 0 "#PWR0164" H 1800 3200 50  0001 C CNN
+F 0 "#PWR060" H 1800 3200 50  0001 C CNN
 F 1 "GND" H 1805 3277 50  0000 C CNN
 F 2 "" H 1800 3450 50  0001 C CNN
@@
 	2300 950  2300 1200
 $Comp
-L Mechanical:MountingHole_Pad H2
+L Mechanical:MountingHole_Pad H6
 U 1 1 5F3A7758
 P 3000 3450
-F 0 "H2" H 3100 3600 50  0000 L CNN
+F 0 "H6" H 3100 3600 50  0000 L CNN
 F 1 "MountingHole_Pad" H 3100 3408 50  0001 L CNN
 F 2 "MountingHole:MountingHole_4.3mm_M4_Pad_Via" H 3000 3450 50  0001 C CNN
@@
 $EndComp
 $Comp
-L Device:C C24
+L Device:C C18
 U 1 1 5F3A7900
 P 3000 3700
-F 0 "C24" H 3115 3746 50  0000 L CNN
+F 0 "C18" H 3115 3746 50  0000 L CNN
 F 1 "1u" H 3115 3655 50  0000 L CNN
 F 2 "Capacitor_SMD:C_1206_3216Metric" H 3038 3550 50  0001 C CNN
@@
 $EndComp
 $Comp
-L power:GND #PWR05
+L power:GND #PWR061
 U 1 1 5F3A972C
 P 3000 3850
-F 0 "#PWR05" H 3000 3600 50  0001 C CNN
+F 0 "#PWR061" H 3000 3600 50  0001 C CNN
 F 1 "GND" H 3005 3677 50  0000 C CNN
 F 2 "" H 3000 3850 50  0001 C CNN
